File: circuit/fortuna-box.kicad_sch (KiCad schematic)
At the start: 6 parts, among them J1 Port B, J2 Port C, J3 Port E, J4 Port A, J5 Port D, J6 Port F

Commit message: .
Other:
- added sheet CPU (cpu.kicad_sch)
- added sheet Debugger (debugger.kicad_sch)
- added sheet Memory (memory.kicad_sch)
- added sheet Serial (serial.kicad_sch)
- added sheet Storage (storage.kicad_sch)
Changed lines of the file:
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@@
+    )
+  )
+  (sheet (at 255.27 22.86) (size 15.875 19.685) (fields_autoplaced)
+    (stroke (width 0.1524) (type solid))
+    (fill (color 0 0 0 0.0000))
+    (property "Sheetname" "Storage" (at 255.27 22.1484 0)
+      (effects (font (size 1.27 1.27)) (justify left bottom))
+    )
+    (property "Sheetfile" "storage.kicad_sch" (at 255.27 43.1296 0)
+      (effects (font (size 1.27 1.27)) (justify left top))
+    )
+    (instances
+      (project "fortuna-box"
+        (path "/0e4c4e8a-78e0-4f49-88dc-754c12656209" (page "5"))
+      )
+    )
+  )
+  (sheet (at 172.085 51.435) (size 16.51 19.685) (fields_autoplaced)
+    (stroke (width 0.1524) (type solid))
+    (fill (color 0 0 0 0.0000))
+    (property "Sheetname" "Debugger" (at 172.085 50.7234 0)
+      (effects (font (size 1.27 1.27)) (justify left bottom))
+    )
+    (property "Sheetfile" "debugger.kicad_sch" (at 172.085 71.7046 0)
+      (effects (font (size 1.27 1.27)) (justify left top))
+    )
+    (instances
+      (project "fortuna-box"
+        (path "/0e4c4e8a-78e0-4f49-88dc-754c12656209" (page "6"))
+      )
+    )
+  )
+  (sheet (at 229.235 22.86) (size 15.24 19.05) (fields_autoplaced)
+    (stroke (width 0.1524) (type solid))
+    (fill (color 0 0 0 0.0000))
+    (property "Sheetname" "Serial" (at 229.235 22.1484 0)
+      (effects (font (size 1.27 1.27)) (justify left bottom))
+    )
+    (property "Sheetfile" "serial.kicad_sch" (at 229.235 42.4946 0)
+      (effects (font (size 1.27 1.27)) (justify left top))
+    )
+    (instances
+      (project "fortuna-box"
+        (path "/0e4c4e8a-78e0-4f49-88dc-754c12656209" (page "4"))
+      )
+    )
+  )
+  (sheet (at 200.025 22.86) (size 15.24 18.415) (fields_autoplaced)
+    (stroke (width 0.1524) (type solid))
+    (fill (color 0 0 0 0.0000))
+    (property "Sheetname" "Memory" (at 200.025 22.1484 0)
+      (effects (font (size 1.27 1.27)) (justify left bottom))
+    )
+    (property "Sheetfile" "memory.kicad_sch" (at 200.025 41.8596 0)
+      (effects (font (size 1.27 1.27)) (justify left top))
+    )
+    (instances
+      (project "fortuna-box"
+        (path "/0e4c4e8a-78e0-4f49-88dc-754c12656209" (page "3"))
+      )
+    )
+  )
+  (sheet (at 172.72 22.86) (size 15.24 17.78) (fields_autoplaced)
+    (stroke (width 0.1524) (type solid))
+    (fill (color 0 0 0 0.0000))
+    (property "Sheetname" "CPU" (at 172.72 22.1484 0)
+      (effects (font (size 1.27 1.27)) (justify left bottom))
+    )
+    (property "Sheetfile" "cpu.kicad_sch" (at 172.72 41.2246 0)
+      (effects (font (size 1.27 1.27)) (justify left top))
+    )
+    (instances
+      (project "fortuna-box"
+        (path "/0e4c4e8a-78e0-4f49-88dc-754c12656209" (page "2"))
+      )
     )
   )

Commit message: .
Parts:
- added J34: Port G, symbol Connector_Generic:Conn_02x03_Counter_Clockwise
Connections:
- new net RX: J34.6 (Pin_6)
- new net TX: J34.5 (Pin_5)
Other:
- added sheet Video (video.kicad_sch)
- note added: "26 holes"
- note added: "37 holes"
- note added: "CPU & debugger: A, B, C, D, E, F, G Memory: A, C, D, E, G Peripherals: A, B, C, G"
- note added: "Leave space for a possible additional Port G"
- note removed: "CPU & debugger: A, B, C, D, E, F Memory: A, C, D, E Peripherals: A, B, C"
Changed lines of the file:
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@@
+    (stroke (width 0) (type default))
+  )
+  (wire (pts (xy 135.89 65.405) (xy 125.095 65.405))
     (stroke (width 0) (type default))
   )
@@
     (stroke (width 0) (type default))
   )
+  (wire (pts (xy 135.89 62.865) (xy 125.095 62.865))
+    (stroke (width 0) (type default))
+  )
   (wire (pts (xy 43.815 38.735) (xy 54.61 38.735))
     (stroke (width 0) (type default))
@@
     (effects (font (size 1.27 1.27)) (justify left bottom))
   )
+  (text "Leave space for\na possible additional\nPort G" (at 100.965 128.27 0)
+    (effects (font (size 1.27 1.27)) (justify left bottom))
+  )
   (text "Port A" (at 41.91 137.795 90)
     (effects (font (size 1.27 1.27)) (justify left bottom))
   )
+  (text "37 holes" (at 36.195 152.4 90)
+    (effects (font (size 1.27 1.27)) (justify left bottom))
+  )
+  (text "26 holes" (at 73.025 183.515 0)
+    (effects (font (size 1.27 1.27)) (justify right bottom))
+  )
   (text "Port B" (at 41.91 151.13 90)
     (effects (font (size 1.27 1.27)) (justify left bottom))
   )
-  (text "CPU & debugger: A, B, C, D, E, F\nMemory: A, C, D, E\nPeripherals: A, B, C\n"
+  (text "CPU & debugger: A, B, C, D, E, F, G\nMemory: A, C, D, E, G\nPeripherals: A, B, C, G\n"
     (at 116.205 51.435 0)
     (effects (font (size 1.27 1.27)) (justify left bottom))
@@
     (effects (font (size 1.27 1.27)) (justify right bottom))
   )
+  (label "RX" (at 135.89 62.865 180) (fields_autoplaced)
+    (effects (font (size 1.27 1.27)) (justify right bottom))
+  )
   (label "A16" (at 132.715 78.105 180) (fields_autoplaced)
     (effects (font (size 1.27 1.27)) (justify right bottom))
@@
   )
   (label "A10" (at 99.695 83.82 180) (fields_autoplaced)
+    (effects (font (size 1.27 1.27)) (justify right bottom))
+  )
+  (label "TX" (at 135.89 65.405 180) (fields_autoplaced)
     (effects (font (size 1.27 1.27)) (justify right bottom))
   )
@@
         (path "/0e4c4e8a-78e0-4f49-88dc-754c12656209"
           (reference "J5") (unit 1)
+        )
+      )
+    )
+  )
+  (symbol (lib_id "Connector_Generic:Conn_02x03_Counter_Clockwise") (at 117.475 65.405 0) (unit 1)
+    (in_bom yes) (on_board yes) (dnp no)
+    (property "Reference" "J34" (at 118.745 56.515 0)
+      (effects (font (size 1.27 1.27)))
+    )
+    (property "Value" "Port G" (at 118.745 59.055 0)
+      (effects (font (size 1.27 1.27)))
+    )
+    (property "Footprint" "" (at 117.475 65.405 0)
+      (effects (font (size 1.27 1.27)) hide)
+    )
+    (property "Datasheet" "~" (at 117.475 65.405 0)
+      (effects (font (size 1.27 1.27)) hide)
+    )
+    (pin "1")
+    (pin "2")
+    (pin "3")
+    (pin "4")
+    (pin "5")
+    (pin "6")
+    (instances
+      (project "fortuna-box"
+        (path "/0e4c4e8a-78e0-4f49-88dc-754c12656209"
+          (reference "J34") (unit 1)
+        )
+        (path "/0e4c4e8a-78e0-4f49-88dc-754c12656209/afd1b413-de30-4838-bb16-3d0c9f3cd196"
+          (reference "J33") (unit 1)
         )
       )
@@
     )
   )
-  (sheet (at 172.085 51.435) (size 16.51 19.685) (fields_autoplaced)
+  (sheet (at 201.295 52.07) (size 13.97 19.685) (fields_autoplaced)
     (stroke (width 0.1524) (type solid))
     (fill (color 0 0 0 0.0000))
-    (property "Sheetname" "Debugger" (at 172.085 50.7234 0)
+    (property "Sheetname" "Debugger" (at 201.295 51.3584 0)
       (effects (font (size 1.27 1.27)) (justify left bottom))
     )
-    (property "Sheetfile" "debugger.kicad_sch" (at 172.085 71.7046 0)
+    (property "Sheetfile" "debugger.kicad_sch" (at 201.295 72.3396 0)
       (effects (font (size 1.27 1.27)) (justify left top))
     )
     (instances
       (project "fortuna-box"
-        (path "/0e4c4e8a-78e0-4f49-88dc-754c12656209" (page "6"))
+        (path "/0e4c4e8a-78e0-4f49-88dc-754c12656209" (page "7"))
       )
     )
@@
       )
     )
+  )
+  (sheet (at 172.72 52.07) (size 15.875 20.32) (fields_autoplaced)
+    (stroke (width 0.1524) (type solid))
+    (fill (color 0 0 0 0.0000))
+    (property "Sheetname" "Video" (at 172.72 51.3584 0)
+      (effects (font (size 1.27 1.27)) (justify left bottom))
+    )
+    (property "Sheetfile" "video.kicad_sch" (at 172.72 72.9746 0)
+      (effects (font (size 1.27 1.27)) (justify left top))
+    )
+    (instances
+      (project "fortuna-box"
+        (path "/0e4c4e8a-78e0-4f49-88dc-754c12656209" (page "6"))
+      )
+    )

Commit message: .
Parts:
- removed J34: Port G, symbol Connector_Generic:Conn_02x03_Counter_Clockwise
- removed J4: Port A, symbol Connector_Generic:Conn_02x03_Counter_Clockwise
- added J4: Port A, symbol Connector_Generic:Conn_01x06
- added J43: Port G, symbol Connector_Generic:Conn_01x06
Connections:
- net A1: now also J4.6 (Pin_6)
- net A2: now also J4.5 (Pin_5)
- net A3: now also J4.4 (Pin_4)
- net GND: now also J4.2 (Pin_2)
- net RX: now also J43.1 (Pin_1)
- net TX: now also J43.2 (Pin_2)
- net VCC: now also J4.1 (Pin_1)
- net ~{RST}: now also J4.3 (Pin_3)
Changed lines of the file:
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@@
     (stroke (width 0) (type default))
   )
-  (wire (pts (xy 78.105 36.195) (xy 67.31 36.195))
-    (stroke (width 0) (type default))
-  )
-  (wire (pts (xy 135.89 65.405) (xy 125.095 65.405))
+  (wire (pts (xy 45.72 31.115) (xy 56.515 31.115))
     (stroke (width 0) (type default))
   )
@@
     (stroke (width 0) (type default))
   )
+  (wire (pts (xy 99.695 28.575) (xy 88.9 28.575))
+    (stroke (width 0) (type default))
+  )
   (wire (pts (xy 99.695 66.675) (xy 88.9 66.675))
     (stroke (width 0) (type default))
   )
-  (wire (pts (xy 43.815 36.195) (xy 54.61 36.195))
+  (wire (pts (xy 45.72 36.195) (xy 56.515 36.195))
+    (stroke (width 0) (type default))
+  )
+  (wire (pts (xy 99.695 26.035) (xy 88.9 26.035))
     (stroke (width 0) (type default))
   )
@@
     (stroke (width 0) (type default))
   )
-  (wire (pts (xy 43.815 33.655) (xy 54.61 33.655))
-    (stroke (width 0) (type default))
-  )
-  (wire (pts (xy 78.105 33.655) (xy 67.31 33.655))
+  (wire (pts (xy 45.72 33.655) (xy 56.515 33.655))
     (stroke (width 0) (type default))
   )
@@
     (stroke (width 0) (type default))
   )
+  (wire (pts (xy 45.72 26.035) (xy 56.515 26.035))
+    (stroke (width 0) (type default))
+  )
   (wire (pts (xy 45.72 81.28) (xy 56.515 81.28))
     (stroke (width 0) (type default))
@@
     (stroke (width 0) (type default))
   )
+  (wire (pts (xy 45.72 28.575) (xy 56.515 28.575))
+    (stroke (width 0) (type default))
+  )
   (wire (pts (xy 99.695 46.355) (xy 88.9 46.355))
     (stroke (width 0) (type default))
@@
     (stroke (width 0) (type default))
   )
-  (wire (pts (xy 135.89 62.865) (xy 125.095 62.865))
-    (stroke (width 0) (type default))
-  )
-  (wire (pts (xy 43.815 38.735) (xy 54.61 38.735))
-    (stroke (width 0) (type default))
-  )
-  (wire (pts (xy 78.105 38.735) (xy 67.31 38.735))
+  (wire (pts (xy 45.72 38.735) (xy 56.515 38.735))
     (stroke (width 0) (type default))
   )
@@
   )
   (text "CPU & debugger: A, B, C, D, E, F, G\nMemory: A, C, D, E, G\nPeripherals: A, B, C, G\n"
-    (at 116.205 51.435 0)
+    (at 114.935 36.83 0)
     (effects (font (size 1.27 1.27)) (justify left bottom))
   )
@@
     (effects (font (size 1.27 1.27)) (justify left bottom))
   )
+  (label "VCC" (at 45.72 26.035 0) (fields_autoplaced)
+    (effects (font (size 1.27 1.27)) (justify left bottom))
+  )
   (label "A13" (at 99.695 91.44 180) (fields_autoplaced)
     (effects (font (size 1.27 1.27)) (justify right bottom))
@@
     (effects (font (size 1.27 1.27)) (justify right bottom))
   )
-  (label "~{RST}" (at 78.105 38.735 180) (fields_autoplaced)
+  (label "TX" (at 99.695 28.575 180) (fields_autoplaced)
     (effects (font (size 1.27 1.27)) (justify right bottom))
   )
@@
     (effects (font (size 1.27 1.27)) (justify right bottom))
   )
-  (label "RX" (at 135.89 62.865 180) (fields_autoplaced)
-    (effects (font (size 1.27 1.27)) (justify right bottom))
-  )
   (label "A16" (at 132.715 78.105 180) (fields_autoplaced)
     (effects (font (size 1.27 1.27)) (justify right bottom))
@@
     (effects (font (size 1.27 1.27)) (justify right bottom))
   )
+  (label "GND" (at 45.72 28.575 0) (fields_autoplaced)
+    (effects (font (size 1.27 1.27)) (justify left bottom))
+  )
   (label "A7" (at 45.72 96.52 0) (fields_autoplaced)
     (effects (font (size 1.27 1.27)) (justify left bottom))
@@
     (effects (font (size 1.27 1.27)) (justify right bottom))
   )
-  (label "TX" (at 135.89 65.405 180) (fields_autoplaced)
-    (effects (font (size 1.27 1.27)) (justify right bottom))
-  )
-  (label "GND" (at 78.105 36.195 180) (fields_autoplaced)
-    (effects (font (size 1.27 1.27)) (justify right bottom))
-  )
   (label "CLK" (at 132.715 98.425 180) (fields_autoplaced)
     (effects (font (size 1.27 1.27)) (justify right bottom))
@@
     (effects (font (size 1.27 1.27)) (justify right bottom))
   )
+  (label "~{RST}" (at 45.72 31.115 0) (fields_autoplaced)
+    (effects (font (size 1.27 1.27)) (justify left bottom))
+  )
   (label "A9" (at 99.695 81.28 180) (fields_autoplaced)
     (effects (font (size 1.27 1.27)) (justify right bottom))
@@
     (effects (font (size 1.27 1.27)) (justify left bottom))
   )
-  (label "A2" (at 43.815 36.195 0) (fields_autoplaced)
-    (effects (font (size 1.27 1.27)) (justify left bottom))
-  )
-  (label "A3" (at 43.815 33.655 0) (fields_autoplaced)
+  (label "RX" (at 99.695 26.035 180) (fields_autoplaced)
+    (effects (font (size 1.27 1.27)) (justify right bottom))
+  )
+  (label "A2" (at 45.72 36.195 0) (fields_autoplaced)
+    (effects (font (size 1.27 1.27)) (justify left bottom))
+  )
+  (label "A3" (at 45.72 33.655 0) (fields_autoplaced)
     (effects (font (size 1.27 1.27)) (justify left bottom))
   )
@@
     (effects (font (size 1.27 1.27)) (justify left bottom))
   )
-  (label "A1" (at 43.815 38.735 0) (fields_autoplaced)
+  (label "A1" (at 45.72 38.735 0) (fields_autoplaced)
     (effects (font (size 1.27 1.27)) (justify left bottom))
   )
@@
     (effects (font (size 1.27 1.27)) (justify left bottom))
   )
-  (label "VCC" (at 78.105 33.655 180) (fields_autoplaced)
-    (effects (font (size 1.27 1.27)) (justify right bottom))
-  )
   (label "~{ROM_WE}" (at 45.72 86.36 0) (fields_autoplaced)
     (effects (font (size 1.27 1.27)) (justify left bottom))
+  )
+  (symbol (lib_id "Connector_Generic:Conn_01x06") (at 83.82 31.115 0) (mirror y) (unit 1)
+    (in_bom yes) (on_board yes) (dnp no)
+    (property "Reference" "J43" (at 80.645 31.115 0)
+      (effects (font (size 1.27 1.27)) (justify left))
+    )
+    (property "Value" "Port G" (at 80.645 33.655 0)
+      (effects (font (size 1.27 1.27)) (justify left))
+    )
+    (property "Footprint" "" (at 83.82 31.115 0)
+      (effects (font (size 1.27 1.27)) hide)
+    )
+    (property "Datasheet" "~" (at 83.82 31.115 0)
+      (effects (font (size 1.27 1.27)) hide)
+    )
+    (pin "1")
+    (pin "2")
+    (pin "3")
+    (pin "4")
+    (pin "5")
+    (pin "6")
+    (instances
+      (project "fortuna-box"
+        (path "/0e4c4e8a-78e0-4f49-88dc-754c12656209"
+          (reference "J43") (unit 1)
+        )
+      )
+    )
   )
   (symbol (lib_id "Connector_Generic:Conn_01x08") (at 61.595 86.36 0) (unit 1)
@@
     )
   )
-  (symbol (lib_id "Connector_Generic:Conn_02x03_Counter_Clockwise") (at 117.475 65.405 0) (unit 1)
-    (in_bom yes) (on_board yes) (dnp no)
-    (property "Reference" "J34" (at 118.745 56.515 0)
-      (effects (font (size 1.27 1.27)))
-    )
-    (property "Value" "Port G" (at 118.745 59.055 0)
-      (effects (font (size 1.27 1.27)))
-    )
-    (property "Footprint" "" (at 117.475 65.405 0)
-      (effects (font (size 1.27 1.27)) hide)
-    )
-    (property "Datasheet" "~" (at 117.475 65.405 0)
-      (effects (font (size 1.27 1.27)) hide)
-    )
-    (pin "1")
-    (pin "2")
-    (pin "3")
-    (pin "4")
-    (pin "5")
-    (pin "6")
-    (instances
-      (project "fortuna-box"
-        (path "/0e4c4e8a-78e0-4f49-88dc-754c12656209"
-          (reference "J34") (unit 1)
-        )
-        (path "/0e4c4e8a-78e0-4f49-88dc-754c12656209/afd1b413-de30-4838-bb16-3d0c9f3cd196"
-          (reference "J33") (unit 1)
-        )
-      )
-    )
-  )
   (symbol (lib_id "Connector_Generic:Conn_01x08") (at 83.82 86.36 0) (mirror y) (unit 1)
     (in_bom yes) (on_board yes) (dnp no)
@@
     )
   )
-  (symbol (lib_id "Connector_Generic:Conn_02x03_Counter_Clockwise") (at 59.69 36.195 0) (unit 1)
-    (in_bom yes) (on_board yes) (dnp no)
-    (property "Reference" "J4" (at 60.96 27.305 0)
-      (effects (font (size 1.27 1.27)))
-    )
-    (property "Value" "Port A" (at 60.96 29.845 0)
-      (effects (font (size 1.27 1.27)))
-    )
-    (property "Footprint" "" (at 59.69 36.195 0)
-      (effects (font (size 1.27 1.27)) hide)
-    )
-    (property "Datasheet" "~" (at 59.69 36.195 0)
-      (effects (font (size 1.27 1.27)) hide)
-    )
+  (symbol (lib_id "Connector_Generic:Conn_01x06") (at 61.595 31.115 0) (unit 1)
+    (in_bom yes) (on_board yes) (dnp no) (fields_autoplaced)
+    (property "Reference" "J4" (at 64.77 31.115 0)
+      (effects (font (size 1.27 1.27)) (justify left))
+    )
+    (property "Value" "Port A" (at 64.77 33.655 0)
+      (effects (font (size 1.27 1.27)) (justify left))
+    )
+    (property "Footprint" "" (at 61.595 31.115 0)
+      (effects (font (size 1.27 1.27)) hide)
+    )
+    (property "Datasheet" "~" (at 61.595 31.115 0)
+      (effects (font (size 1.27 1.27)) hide)
+    )
