File: circuit/fortuna-box.kicad_sch (KiCad schematic)
At the start: 7 parts, among them J1 Port B, J2 Port C, J3 Port E, J4 Port A, J43 Port G, J5 Port D, J6 Port F

Commit message: .
Parts:
- removed J6: Port F, symbol Connector_Generic:Conn_01x10
- added J14: Port F, symbol Connector_Generic:Conn_01x08
Connections:
- net A16: now also J43.4 (Pin_4)
- net A17: now also J43.5 (Pin_5)
- net A18: now also J43.6 (Pin_6)
- net CLK: now also J14.7 (Pin_7)
- net CLK_ENA: now also J14.8 (Pin_8)
- net ~{BUSAK}: now also J14.3 (Pin_3)
- net ~{BUSRQ}: now also J14.2 (Pin_2)
- net ~{IORQ}: now also J14.6 (Pin_6)
- net ~{M1}: now also J14.5 (Pin_5)
- net ~{NMI}: now also J14.4 (Pin_4)
- net RAMONLY: now reaches J43.3 (Pin_3)
- no-connect marks 0 -> 1
Changed lines of the file:
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@@
 (kicad_sch (version 20230121) (generator eeschema)
   (paper "A4")
+  (no_connect (at 121.92 83.185))
   (wire (pts (xy 99.695 59.055) (xy 88.9 59.055))
     (stroke (width 0) (type default))
@@
     (stroke (width 0) (type default))
   )
+  (wire (pts (xy 99.695 38.735) (xy 88.9 38.735))
+    (stroke (width 0) (type default))
+  )
   (wire (pts (xy 99.695 86.36) (xy 88.9 86.36))
     (stroke (width 0) (type default))
   )
+  (wire (pts (xy 99.695 33.655) (xy 88.9 33.655))
+    (stroke (width 0) (type default))
+  )
   (wire (pts (xy 45.72 88.9) (xy 56.515 88.9))
     (stroke (width 0) (type default))
@@
     (stroke (width 0) (type default))
   )
-  (wire (pts (xy 132.715 80.645) (xy 121.92 80.645))
-    (stroke (width 0) (type default))
-  )
   (wire (pts (xy 99.695 61.595) (xy 88.9 61.595))
     (stroke (width 0) (type default))
@@
     (stroke (width 0) (type default))
   )
-  (wire (pts (xy 132.715 83.185) (xy 121.92 83.185))
+  (wire (pts (xy 88.9 31.115) (xy 99.695 31.115))
     (stroke (width 0) (type default))
   )
@@
     (stroke (width 0) (type default))
   )
+  (wire (pts (xy 99.695 36.195) (xy 88.9 36.195))
+    (stroke (width 0) (type default))
+  )
   (wire (pts (xy 45.72 53.975) (xy 56.515 53.975))
     (stroke (width 0) (type default))
@@
   )
   (wire (pts (xy 45.72 91.44) (xy 56.515 91.44))
-    (stroke (width 0) (type default))
-  )
-  (wire (pts (xy 132.715 78.105) (xy 121.92 78.105))
     (stroke (width 0) (type default))
   )
@@
     (effects (font (size 1.27 1.27)) (justify right bottom))
   )
+  (label "A16" (at 99.695 33.655 180) (fields_autoplaced)
+    (effects (font (size 1.27 1.27)) (justify right bottom))
+  )
   (label "~{IORQ}" (at 132.715 95.885 180) (fields_autoplaced)
     (effects (font (size 1.27 1.27)) (justify right bottom))
@@
     (effects (font (size 1.27 1.27)) (justify right bottom))
   )
+  (label "A17" (at 99.695 36.195 180) (fields_autoplaced)
+    (effects (font (size 1.27 1.27)) (justify right bottom))
+  )
   (label "A0" (at 99.695 69.215 180) (fields_autoplaced)
     (effects (font (size 1.27 1.27)) (justify right bottom))
@@
     (effects (font (size 1.27 1.27)) (justify right bottom))
   )
-  (label "A16" (at 132.715 78.105 180) (fields_autoplaced)
-    (effects (font (size 1.27 1.27)) (justify right bottom))
-  )
   (label "Y2W" (at 45.72 56.515 0) (fields_autoplaced)
     (effects (font (size 1.27 1.27)) (justify left bottom))
@@
     (effects (font (size 1.27 1.27)) (justify left bottom))
   )
-  (label "A17" (at 132.715 80.645 180) (fields_autoplaced)
-    (effects (font (size 1.27 1.27)) (justify right bottom))
-  )
   (label "D6" (at 99.695 61.595 180) (fields_autoplaced)
     (effects (font (size 1.27 1.27)) (justify right bottom))
@@
     (effects (font (size 1.27 1.27)) (justify left bottom))
   )
-  (label "A18" (at 132.715 83.185 180) (fields_autoplaced)
+  (label "RAMONLY" (at 99.695 31.115 180) (fields_autoplaced)
     (effects (font (size 1.27 1.27)) (justify right bottom))
   )
@@
   (label "A5" (at 45.72 91.44 0) (fields_autoplaced)
     (effects (font (size 1.27 1.27)) (justify left bottom))
+  )
+  (label "A18" (at 99.695 38.735 180) (fields_autoplaced)
+    (effects (font (size 1.27 1.27)) (justify right bottom))
   )
   (label "A6" (at 45.72 93.98 0) (fields_autoplaced)
@@
         (path "/0e4c4e8a-78e0-4f49-88dc-754c12656209"
           (reference "J43") (unit 1)
+        )
+      )
+    )
+  )
+  (symbol (lib_id "Connector_Generic:Conn_01x08") (at 116.84 90.805 0) (mirror y) (unit 1)
+    (in_bom yes) (on_board yes) (dnp no)
+    (property "Reference" "J14" (at 114.3 90.805 0)
+      (effects (font (size 1.27 1.27)) (justify left))
+    )
+    (property "Value" "Port F" (at 114.3 93.345 0)
+      (effects (font (size 1.27 1.27)) (justify left))
+    )
+    (property "Footprint" "" (at 116.84 90.805 0)
+      (effects (font (size 1.27 1.27)) hide)
+    )
+    (property "Datasheet" "~" (at 116.84 90.805 0)
+      (effects (font (size 1.27 1.27)) hide)
+    )
+    (pin "1")
+    (pin "2")
+    (pin "3")
+    (pin "4")
+    (pin "5")
+    (pin "6")
+    (pin "7")
+    (pin "8")
+    (instances
+      (project "fortuna-box"
+        (path "/0e4c4e8a-78e0-4f49-88dc-754c12656209"
+          (reference "J14") (unit 1)
+        )
+        (path "/0e4c4e8a-78e0-4f49-88dc-754c12656209/afd1b413-de30-4838-bb16-3d0c9f3cd196"
+          (reference "J12") (unit 1)
+        )
+        (path "/0e4c4e8a-78e0-4f49-88dc-754c12656209/34f47b44-6e82-4397-9bc8-849df4113da9"
+          (reference "J13") (unit 1)
         )
       )
@@
         )
       )
-    )
-  )
-  (symbol (lib_id "Connector_Generic:Conn_01x10") (at 116.84 88.265 0) (mirror y) (unit 1)
-    (in_bom yes) (on_board yes) (dnp no)
-    (property "Reference" "J6" (at 113.665 88.265 0)
-      (effects (font (size 1.27 1.27)) (justify left))
-    )
-    (property "Value" "Port F" (at 113.665 90.805 0)
-      (effects (font (size 1.27 1.27)) (justify left))
-    )
-    (property "Footprint" "" (at 116.84 88.265 0)
-      (effects (font (size 1.27 1.27)) hide)
-    )
-    (property "Datasheet" "~" (at 116.84 88.265 0)
-      (effects (font (size 1.27 1.27)) hide)
-    )
-    (pin "1")
-    (pin "10")
-    (pin "2")
-    (pin "3")
-    (pin "4")
-    (pin "5")
-    (pin "6")
-    (pin "7")
-    (pin "8")
-    (pin "9")
-    (instances
-      (project "fortuna-box"
-        (path "/0e4c4e8a-78e0-4f49-88dc-754c12656209"
-          (reference "J6") (unit 1)
-        )
-      )

Commit message: .
Other:
- added sheet Power (power.kicad_sch)
Changed lines of the file:
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@@
+    )
+  )
+  (sheet (at 229.87 53.34) (size 13.97 19.05) (fields_autoplaced)
+    (stroke (width 0.1524) (type solid))
+    (fill (color 0 0 0 0.0000))
+    (property "Sheetname" "Power" (at 229.87 52.6284 0)
+      (effects (font (size 1.27 1.27)) (justify left bottom))
+    )
+    (property "Sheetfile" "power.kicad_sch" (at 229.87 72.9746 0)
+      (effects (font (size 1.27 1.27)) (justify left top))
+    )
+    (instances
+      (project "fortuna-box"
+        (path "/0e4c4e8a-78e0-4f49-88dc-754c12656209" (page "8"))
+      )
     )
   )

Commit message: .
Connections:
- net RAMONLY: now also J14.6 (Pin_6); no longer J43.3 (Pin_3)
- net ~{IORQ}: now also J43.3 (Pin_3); no longer J14.6 (Pin_6)
Other:
- note added: "CPU & debugger: A, B, C, D, E, F, G Memory: A, C, D, E, F, G Peripherals: A, B, C, G"
- note removed: "CPU & debugger: A, B, C, D, E, F, G Memory: A, C, D, E, G Peripherals: A, B, C, G"
- note removed: "TODO: RX, TX?"
Changed lines of the file:
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@@
     (effects (font (size 1.27 1.27)) (justify right bottom))
-  )
-  (text "TODO: RX, TX?" (at 131.445 106.68 0)
-    (effects (font (size 1.27 1.27)) (justify left bottom))
   )
   (text "Leave space for\na possible additional\nPort G" (at 100.965 128.27 0)
@@
     (effects (font (size 1.27 1.27)) (justify left bottom))
   )
-  (text "CPU & debugger: A, B, C, D, E, F, G\nMemory: A, C, D, E, G\nPeripherals: A, B, C, G\n"
+  (text "CPU & debugger: A, B, C, D, E, F, G\nMemory: A, C, D, E, F, G\nPeripherals: A, B, C, G\n"
     (at 114.935 36.83 0)
     (effects (font (size 1.27 1.27)) (justify left bottom))
@@
     (effects (font (size 1.27 1.27)) (justify right bottom))
   )
-  (label "~{IORQ}" (at 132.715 95.885 180) (fields_autoplaced)
+  (label "RAMONLY" (at 132.715 95.885 180) (fields_autoplaced)
     (effects (font (size 1.27 1.27)) (justify right bottom))
   )
@@
     (effects (font (size 1.27 1.27)) (justify left bottom))
   )
-  (label "RAMONLY" (at 99.695 31.115 180) (fields_autoplaced)
+  (label "~{IORQ}" (at 99.695 31.115 180) (fields_autoplaced)
     (effects (font (size 1.27 1.27)) (justify right bottom))
   )

Commit message: .
Connections:
- net CLK_ENA: no longer names the net of J14.8 (Pin_8)
- no-connect marks 1 -> 2
Other:
- removed sheet Power
- moved on the sheet: J14
Changed lines of the file:
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@@
 (kicad_sch (version 20230121) (generator eeschema)
   (paper "A4")
-  (no_connect (at 121.92 83.185))
+  (no_connect (at 121.92 101.6))
+  (no_connect (at 121.92 83.82))
   (wire (pts (xy 99.695 59.055) (xy 88.9 59.055))
     (stroke (width 0) (type default))
@@
     (stroke (width 0) (type default))
   )
-  (wire (pts (xy 132.715 100.965) (xy 121.92 100.965))
-    (stroke (width 0) (type default))
-  )
   (wire (pts (xy 45.72 33.655) (xy 56.515 33.655))
     (stroke (width 0) (type default))
@@
     (stroke (width 0) (type default))
   )
-  (wire (pts (xy 132.715 95.885) (xy 121.92 95.885))
+  (wire (pts (xy 132.715 96.52) (xy 121.92 96.52))
     (stroke (width 0) (type default))
   )
@@
     (stroke (width 0) (type default))
   )
-  (wire (pts (xy 132.715 93.345) (xy 121.92 93.345))
+  (wire (pts (xy 132.715 93.98) (xy 121.92 93.98))
     (stroke (width 0) (type default))
   )
@@
     (stroke (width 0) (type default))
   )
-  (wire (pts (xy 132.715 98.425) (xy 121.92 98.425))
-    (stroke (width 0) (type default))
-  )
-  (wire (pts (xy 132.715 85.725) (xy 121.92 85.725))
+  (wire (pts (xy 132.715 99.06) (xy 121.92 99.06))
+    (stroke (width 0) (type default))
+  )
+  (wire (pts (xy 132.715 86.36) (xy 121.92 86.36))
     (stroke (width 0) (type default))
   )
@@
     (stroke (width 0) (type default))
   )
-  (wire (pts (xy 132.715 90.805) (xy 121.92 90.805))
+  (wire (pts (xy 132.715 91.44) (xy 121.92 91.44))
     (stroke (width 0) (type default))
   )
@@
     (stroke (width 0) (type default))
   )
-  (wire (pts (xy 132.715 88.265) (xy 121.92 88.265))
+  (wire (pts (xy 132.715 88.9) (xy 121.92 88.9))
     (stroke (width 0) (type default))
   )
@@
     (effects (font (size 1.27 1.27)) (justify right bottom))
   )
-  (label "~{BUSAK}" (at 132.715 88.265 180) (fields_autoplaced)
+  (label "~{BUSAK}" (at 132.715 88.9 180) (fields_autoplaced)
     (effects (font (size 1.27 1.27)) (justify right bottom))
   )
@@
     (effects (font (size 1.27 1.27)) (justify right bottom))
   )
-  (label "RAMONLY" (at 132.715 95.885 180) (fields_autoplaced)
+  (label "RAMONLY" (at 132.715 96.52 180) (fields_autoplaced)
     (effects (font (size 1.27 1.27)) (justify right bottom))
   )
@@
     (effects (font (size 1.27 1.27)) (justify right bottom))
   )
-  (label "~{NMI}" (at 132.715 90.805 180) (fields_autoplaced)
+  (label "~{NMI}" (at 132.715 91.44 180) (fields_autoplaced)
     (effects (font (size 1.27 1.27)) (justify right bottom))
   )
@@
     (effects (font (size 1.27 1.27)) (justify right bottom))
   )
-  (label "~{BUSRQ}" (at 132.715 85.725 180) (fields_autoplaced)
+  (label "~{BUSRQ}" (at 132.715 86.36 180) (fields_autoplaced)
     (effects (font (size 1.27 1.27)) (justify right bottom))
   )
@@
     (effects (font (size 1.27 1.27)) (justify right bottom))
   )
-  (label "~{M1}" (at 132.715 93.345 180) (fields_autoplaced)
+  (label "~{M1}" (at 132.715 93.98 180) (fields_autoplaced)
     (effects (font (size 1.27 1.27)) (justify right bottom))
   )
@@
     (effects (font (size 1.27 1.27)) (justify right bottom))
   )
-  (label "CLK" (at 132.715 98.425 180) (fields_autoplaced)
+  (label "CLK" (at 132.715 99.06 180) (fields_autoplaced)
     (effects (font (size 1.27 1.27)) (justify right bottom))
   )
@@
   (label "Y3W" (at 45.72 61.595 0) (fields_autoplaced)
     (effects (font (size 1.27 1.27)) (justify left bottom))
-  )
-  (label "CLK_ENA" (at 132.715 100.965 180) (fields_autoplaced)
-    (effects (font (size 1.27 1.27)) (justify right bottom))
   )
   (label "Y0W" (at 45.72 46.355 0) (fields_autoplaced)
@@
     )
   )
-  (symbol (lib_id "Connector_Generic:Conn_01x08") (at 116.84 90.805 0) (mirror y) (unit 1)
+  (symbol (lib_id "Connector_Generic:Conn_01x08") (at 116.84 91.44 0) (mirror y) (unit 1)
     (in_bom yes) (on_board yes) (dnp no)
-    (property "Reference" "J14" (at 114.3 90.805 0)
-      (effects (font (size 1.27 1.27)) (justify left))
-    )
-    (property "Value" "Port F" (at 114.3 93.345 0)
-      (effects (font (size 1.27 1.27)) (justify left))
-    )
-    (property "Footprint" "" (at 116.84 90.805 0)
-      (effects (font (size 1.27 1.27)) hide)
-    )
-    (property "Datasheet" "~" (at 116.84 90.805 0)
+    (property "Reference" "J14" (at 114.3 91.44 0)
+      (effects (font (size 1.27 1.27)) (justify left))
+    )
+    (property "Value" "Port F" (at 114.3 93.98 0)
+      (effects (font (size 1.27 1.27)) (justify left))
+    )
+    (property "Footprint" "" (at 116.84 91.44 0)
+      (effects (font (size 1.27 1.27)) hide)
+    )
+    (property "Datasheet" "~" (at 116.84 91.44 0)
       (effects (font (size 1.27 1.27)) hide)
     )
@@
       )
     )
-  )
-  (sheet (at 229.87 53.34) (size 13.97 19.05) (fields_autoplaced)
-    (stroke (width 0.1524) (type solid))
-    (fill (color 0 0 0 0.0000))
-    (property "Sheetname" "Power" (at 229.87 52.6284 0)
-      (effects (font (size 1.27 1.27)) (justify left bottom))
-    )
-    (property "Sheetfile" "power.kicad_sch" (at 229.87 72.9746 0)
-      (effects (font (size 1.27 1.27)) (justify left top))
-    )
-    (instances
-      (project "fortuna-box"
-        (path "/0e4c4e8a-78e0-4f49-88dc-754c12656209" (page "8"))
-      )
-    )
