File: circuit/memory.kicad_sch (KiCad schematic)
At the start: 23 parts, among them J2 Port C, J3 Port E, J4 Port A, J5 Port D, U2 74HTC175

Commit message: .
Parts:
- removed U? (x2): 74LS32, symbol 74xx:74LS32
- added D2 (x3): 1N4148, Diode_THT:D_DO-35_SOD27_P7.62mm_Horizontal, symbol Diode:1N4148
- added J4: Port G, symbol Connector_Generic:Conn_02x03_Counter_Clockwise
- added R?: 10K, symbol Device:R_US
Connections:
- net A13: now also D2.2 (A)
- net A14: now also D2.2 (A)
- net A15: now also D2.2 (A)
- net GND: now also R?.1
- net ~{BOTTOM 8K}: now also U?.12, D2.1 (K), D2.1 (K), D2.1 (K), R?.2
- new net RX: J4.6 (Pin_6)
- new net TX: J4.5 (Pin_5)
Other:
- note added: "OR gate"

Commit message: .
Parts:
- removed J4: Port A, symbol Connector_Generic:Conn_02x03_Counter_Clockwise
- removed J4: Port G, symbol Connector_Generic:Conn_02x03_Counter_Clockwise
- added J4: Port A, symbol Connector_Generic:Conn_01x06
- added J43: Port G, symbol Connector_Generic:Conn_01x06
Connections:
- net A1: now also J4.6 (Pin_6)
- net A2: now also J4.5 (Pin_5)
- net A3: now also J4.4 (Pin_4)
- net GND: now also J4.2 (Pin_2)
- net RX: now also J43.1 (Pin_1)
- net TX: now also J43.2 (Pin_2)
- net VCC: now also J4.1 (Pin_1)
- net ~{RST}: now also J4.3 (Pin_3)
