File: circuit/serial.kicad_sch (KiCad schematic)
At the start: 5 parts

Commit message: .
Parts:
- removed J?: FTDI cable, symbol Connector_Generic:Conn_01x06
- removed R?: 3k3, symbol Device:R_US
- removed U?: 74HCT04, symbol 74xx:74HCT04
- added D13, D14: LED, symbol Device:LED
- added D2 (x2): 1N4148, Diode_THT:D_DO-35_SOD27_P7.62mm_Horizontal, symbol Diode:1N4148
- added J1: Port B, symbol Connector_Generic:Conn_01x10
- added J2: Port C, symbol Connector_Generic:Conn_01x10
- added J4: Port A, symbol Connector_Generic:Conn_02x03_Counter_Clockwise
- added J4: Port G, symbol Connector_Generic:Conn_02x03_Counter_Clockwise
- added J?: FTDI cable, symbol Connector_Generic:Conn_01x06
- added Q1: 2N3904, Package_TO_SOT_THT:TO-92_Inline, symbol Transistor_BJT:2N3904
- added Q2, Q3: 2N3906, Package_TO_SOT_THT:TO-92_Inline, symbol Transistor_BJT:2N3906
- added R? (x2): 220, symbol Device:R_US
- added R? (x2): 43k, symbol Device:R_US
- added R?: 1K, symbol Device:R_US
- added R? (x2): 10k, symbol Device:R_US
Connections:
- net A7 is gone; now on net VCC: U?.10 (CS1)
- net ~{M1} is gone; now on net VCC: U?.8 (CS0)
- net A0: now also J2.10 (Pin_10); no longer U?.11 (RS)
- net CLK_EXT: now also J1.9 (Pin_9)
- net CTS: now also J?.2 (Pin_2)
- net DTR: now also J?.6 (Pin_6)
- net GND: now also J4.5 (Pin_5), J?.1 (Pin_1), Q1.1 (E), R?.2, R?.2
- net RX: now also J4.6 (Pin_6), J?.5 (Pin_5), R?.2
- net TX: now also J4.5 (Pin_5), J?.4 (Pin_4), R?.2
- net VCC: now also J4.6 (Pin_6), J?.3 (Pin_3), Q2.1 (E), Q3.1 (E), R?.1, R?.1
- net ~{INT}: now also J2.9 (Pin_9)
- net ~{IORQ}: now also R?.2
- net at U?.14 (E): now also Q1.3 (C), R?.2
- net A6: no longer names the net of U?.9 (~{CS2})
- net A6: now also D2.2 (A), D2.2 (A), R?.2
- net ~{WR} renamed Y0W
- net Y0W: now also D2.1 (K), J1.1 (Pin_1)
- new net: D13.1 (K), R?.1
- new net: D13.2 (A), Q2.3 (C)
- new net: D14.1 (K), R?.1
- new net: Q1.2 (B), R?.1
- new net: Q3.2 (B), R?.1
- new net: D14.2 (A), Q3.3 (C)
- new net: Q2.2 (B), R?.1
- new net A1: J4.3 (Pin_3)
- new net A2: J4.2 (Pin_2), U?.11 (RS)
- new net A3: J4.1 (Pin_1)
- new net D0: J2.1 (Pin_1)
- new net D1: J2.2 (Pin_2)
- new net D2: J2.3 (Pin_3)
- new net D3: J2.4 (Pin_4)
- new net D4: J2.5 (Pin_5)
- new net D5: J2.6 (Pin_6)
- new net D6: J2.7 (Pin_7)
- new net D7: J2.8 (Pin_8)
- new net Y0R: D2.1 (K), J1.2 (Pin_2)
- new net Y1R: J1.4 (Pin_4)
- new net Y1W: J1.3 (Pin_3)
- new net Y2R: J1.6 (Pin_6)
- new net Y2W: J1.5 (Pin_5)
- new net Y3R: J1.8 (Pin_8)
- new net Y3W: J1.7 (Pin_7)
- new net ~{RST}: J4.4 (Pin_4)
- new net ~{WAIT}: J1.10 (Pin_10)
Other:
- note added: "0x00 - Write config 0x01 - Read status 0x04 - Write to serial 0x05 - Read from serial"
- note added: "A6, A7"
- note added: "Connection Ports"
- note added: "NOT gate"
- note added: "UART indicator lights"
- note removed: "0x80 - Write serial 0x81 - Read serial"
- note removed: "Occupies 0x80 to 0xBF in memory map."
- moved on the sheet: U?

Commit message: .
Parts:
- removed J4: Port A, symbol Connector_Generic:Conn_02x03_Counter_Clockwise
- removed J4: Port G, symbol Connector_Generic:Conn_02x03_Counter_Clockwise
- added J4: Port A, symbol Connector_Generic:Conn_01x06
- added J43: Port G, symbol Connector_Generic:Conn_01x06
Connections:
- net A1: now also J4.6 (Pin_6)
- net A2: now also J4.5 (Pin_5)
- net A3: now also J4.4 (Pin_4)
- net GND: now also J4.2 (Pin_2)
- net RX: now also J43.1 (Pin_1)
- net TX: now also J43.2 (Pin_2)
- net VCC: now also J4.1 (Pin_1)
- net ~{RST}: now also J4.3 (Pin_3)
Other:
- moved on the sheet: J1, J2
