File: circuit/serial.kicad_sch (KiCad schematic)
At the start: 21 parts, among them J1 Port B, J2 Port C, J4 Port A, J43 Port G, Q1 2N3904, Q2 2N3906, Q3 2N3906

Commit message: .
Parts:
- removed Q1: 2N3904, Package_TO_SOT_THT:TO-92_Inline, symbol Transistor_BJT:2N3904
- removed R?: 1K, symbol Device:R_US
- removed R?: 10k, symbol Device:R_US
- added C1: 10uF, symbol Device:C
- added U7: 74HC04, symbol 74xx:74HC04
Connections:
- net GND: now also C1.2
- net VCC: now also C1.1
- net ~{IORQ}: now also U7.1
- net at U?.14 (E): now also U7.2
- net RAMONLY: now reaches J43.3 (Pin_3)
- net A16: now reaches J43.4 (Pin_4)
- net A17: now reaches J43.5 (Pin_5)
- net A18: now reaches J43.6 (Pin_6)
Other:
- note removed: "A6, A7"
- note removed: "NOT gate"

Commit message: .
Connections:
- net RAMONLY renamed ~{RAMONLY}
Changed lines of the file:
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@@
+    (effects (font (size 1.27 1.27)) (justify right bottom))
+  )
+  (label "~{RAMONLY}" (at 261.62 38.1 180) (fields_autoplaced)
     (effects (font (size 1.27 1.27)) (justify right bottom))
   )
@@
     (effects (font (size 1.27 1.27)) (justify left bottom))
   )
-  (label "RAMONLY" (at 261.62 38.1 180) (fields_autoplaced)
-    (effects (font (size 1.27 1.27)) (justify right bottom))
-  )
   (label "D6" (at 261.62 66.04 180) (fields_autoplaced)

Commit message: .
Connections:
- net ~{RAMONLY} is gone; now on net ~{IORQ}: J43.3 (Pin_3)
Changed lines of the file:
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@@
     (effects (font (size 1.27 1.27)) (justify right bottom))
   )
-  (label "~{RAMONLY}" (at 261.62 38.1 180) (fields_autoplaced)
+  (label "~{IORQ}" (at 261.62 38.1 180) (fields_autoplaced)
     (effects (font (size 1.27 1.27)) (justify right bottom))
   )

Commit message: .
Parts:
- D13: value LED -> LED GREEN
- D14: value LED -> LED RED
- R?: value 220 -> 2K
Other:
- note added: "TODO - these transistors might not be necessary, the 74HC04 might drive these LEDs."
Changed lines of the file:
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@@
     (effects (font (size 3 3) (thickness 0.6) bold) (justify left bottom))
+  )
+  (text "TODO - these transistors might not\nbe necessary, the 74HC04 might drive\nthese LEDs."
+    (at 135.89 149.86 0)
+    (effects (font (size 1 1) italic) (justify left bottom))
   )
   (label "Y3R" (at 208.915 68.58 0) (fields_autoplaced)
@@
   (symbol (lib_id "Device:LED") (at 72.39 156.21 90) (unit 1)
     (in_bom yes) (on_board yes) (dnp no) (fields_autoplaced)
-    (property "Reference" "D13" (at 75.565 156.5275 90)
-      (effects (font (size 1.27 1.27)) (justify right))
-    )
-    (property "Value" "LED" (at 75.565 159.0675 90)
+    (property "Reference" "D13" (at 76.2 156.5275 90)
+      (effects (font (size 1.27 1.27)) (justify right))
+    )
+    (property "Value" "LED GREEN" (at 76.2 159.0675 90)
       (effects (font (size 1.27 1.27)) (justify right))
     )
@@
       (effects (font (size 1.27 1.27)) (justify right))
     )
-    (property "Value" "220" (at 69.85 162.5601 0)
+    (property "Value" "2K" (at 69.85 162.5601 0)
       (effects (font (size 1.27 1.27)) (justify right))
     )
@@
   (symbol (lib_id "Device:LED") (at 118.11 156.845 90) (unit 1)
     (in_bom yes) (on_board yes) (dnp no) (fields_autoplaced)
-    (property "Reference" "D14" (at 121.285 157.1625 90)
-      (effects (font (size 1.27 1.27)) (justify right))
-    )
-    (property "Value" "LED" (at 121.285 159.7025 90)
-      (effects (font (size 1.27 1.27)) (justify right))
-    )
+    (property "Reference" "D14" (at 121.92 157.1625 90)
+      (effects (font (size 1.27 1.27)) (justify right))
+    )
+    (property "Value" "LED RED" (at 121.92 159.7025 90)
+      (effects (font (size 1.27 1.27)) (justify right))
+    )

Commit message: .
Connections:
- net Y0R: no longer D2.1 (K)
- net Y0W: no longer D2.1 (K), U?.13 (R/~{W})
- net Y1R: now also D2.1 (K)
- net Y1W: now also D2.1 (K), U?.13 (R/~{W})
Other:
- note added: "0x01 W - Write config 0x01 R - Read status 0x05 W - Write to serial 0x05 R - Read from serial"
- note removed: "0x00 - Write config 0x01 - Read status 0x04 - Write to serial 0x05 - Read from serial"
Changed lines of the file:
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@@
     (effects (font (size 1.27 1.27) italic) (justify left bottom))
   )
-  (text "0x00 - Write config\n0x01 - Read status\n0x04 - Write to serial\n0x05 - Read from serial"
+  (text "0x01 W - Write config\n0x01 R - Read status\n0x05 W - Write to serial\n0x05 R - Read from serial"
     (at 33.655 50.165 0)
     (effects (font (size 1.27 1.27)) (justify left bottom))
@@
     (effects (font (size 1.27 1.27)) (justify right bottom))
   )
-  (label "Y0R" (at 50.8 61.595 0) (fields_autoplaced)
+  (label "Y1R" (at 50.8 61.595 0) (fields_autoplaced)
     (effects (font (size 1.27 1.27)) (justify left bottom))
   )
@@
     (effects (font (size 1.27 1.27)) (justify right bottom))
   )
-  (label "Y0W" (at 86.995 69.215 0) (fields_autoplaced)
+  (label "Y1W" (at 86.995 69.215 0) (fields_autoplaced)
     (effects (font (size 1.27 1.27)) (justify left bottom))
   )
@@
     (effects (font (size 1.27 1.27)) (justify right bottom))
   )
-  (label "Y0W" (at 50.8 66.04 0) (fields_autoplaced)
+  (label "Y1W" (at 50.8 66.04 0) (fields_autoplaced)
     (effects (font (size 1.27 1.27)) (justify left bottom))
   )

Commit message: .
Connections:
- net RX: now also U?.6 (Tx_Data); no longer U?.2 (Rx_Data)
- net TX: now also U?.2 (Rx_Data); no longer U?.6 (Tx_Data)
Other:
- moved on the sheet: D2, J?, R?, U7A, U?

Commit message: .
Parts:
- removed D13: LED GREEN, symbol Device:LED
- removed D14: LED RED, symbol Device:LED
- removed Q2, Q3: 2N3906, Package_TO_SOT_THT:TO-92_Inline, symbol Transistor_BJT:2N3906
- removed R?: 220, symbol Device:R_US
- removed R? (x2): 43k, symbol Device:R_US
- removed R?: 2K, symbol Device:R_US
- added D1: LED GREEN, symbol Device:LED
- added D3: LED RED, symbol Device:LED
- added R?: 220, symbol Device:R_US
- added R?: 2K, symbol Device:R_US
- added U6: 74HC04, symbol 74xx:74HC04
- added unit 3 of U7
Connections:
- net GND: now also R?.2, R?.2
- net RX: now also U6.3
- net TX: now also U7.5
- new net: D3.1 (K), R?.1
- new net: D1.1 (K), R?.1
- new net: D1.2 (A), U6.4
- new net: D3.2 (A), U7.6
Other:
- note removed: "TODO - these transistors might not be necessary, the 74HC04 might drive these LEDs."
