File: circuit/serial.kicad_sch (KiCad schematic)
At the start: 17 parts, among them J1 Port B, J2 Port C, J4 Port A, J43 Port G, U6 74HC04, U7 74HC04

Commit message: .
Parts:
- renumbered J4 to J19, J1 to J20, J2 to J21, J43 to J35
Changed lines of the file:
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@@
       )
       (project "fortuna-box"
-        (path "/0e4c4e8a-78e0-4f49-88dc-754c12656209/afd1b413-de30-4838-bb16-3d0c9f3cd196"
-          (reference "D4") (unit 1)
-        )
         (path "/0e4c4e8a-78e0-4f49-88dc-754c12656209/4037b4b4-0005-458e-a3e9-fe2ae826ab0c"
           (reference "D12") (unit 1)
@@
       )
       (project "fortuna-box"
-        (path "/0e4c4e8a-78e0-4f49-88dc-754c12656209/afd1b413-de30-4838-bb16-3d0c9f3cd196"
-          (reference "D4") (unit 1)
-        )
         (path "/0e4c4e8a-78e0-4f49-88dc-754c12656209/4037b4b4-0005-458e-a3e9-fe2ae826ab0c"
           (reference "D11") (unit 1)
@@
   (symbol (lib_id "Connector_Generic:Conn_01x10") (at 224.79 60.96 0) (unit 1)
     (in_bom yes) (on_board yes) (dnp no) (fields_autoplaced)
-    (property "Reference" "J1" (at 227.965 60.96 0)
+    (property "Reference" "J20" (at 227.965 60.96 0)
       (effects (font (size 1.27 1.27)) (justify left))
     )
@@
     (instances
       (project "fortuna-box"
-        (path "/0e4c4e8a-78e0-4f49-88dc-754c12656209"
-          (reference "J1") (unit 1)
-        )
         (path "/0e4c4e8a-78e0-4f49-88dc-754c12656209/4037b4b4-0005-458e-a3e9-fe2ae826ab0c"
           (reference "J20") (unit 1)
@@
       )
       (project "fortuna-box"
-        (path "/0e4c4e8a-78e0-4f49-88dc-754c12656209/afd1b413-de30-4838-bb16-3d0c9f3cd196"
-          (reference "R13") (unit 1)
-        )
         (path "/0e4c4e8a-78e0-4f49-88dc-754c12656209/4037b4b4-0005-458e-a3e9-fe2ae826ab0c"
           (reference "R8") (unit 1)
@@
   (symbol (lib_id "Connector_Generic:Conn_01x06") (at 245.745 38.1 0) (mirror y) (unit 1)
     (in_bom yes) (on_board yes) (dnp no)
-    (property "Reference" "J43" (at 242.57 38.1 0)
+    (property "Reference" "J35" (at 242.57 38.1 0)
       (effects (font (size 1.27 1.27)) (justify left))
     )
@@
     (instances
       (project "fortuna-box"
-        (path "/0e4c4e8a-78e0-4f49-88dc-754c12656209"
-          (reference "J43") (unit 1)
-        )
-        (path "/0e4c4e8a-78e0-4f49-88dc-754c12656209/afd1b413-de30-4838-bb16-3d0c9f3cd196"
-          (reference "J33") (unit 1)
-        )
         (path "/0e4c4e8a-78e0-4f49-88dc-754c12656209/4037b4b4-0005-458e-a3e9-fe2ae826ab0c"
           (reference "J35") (unit 1)
@@
       )
       (project "fortuna-box"
-        (path "/0e4c4e8a-78e0-4f49-88dc-754c12656209/afd1b413-de30-4838-bb16-3d0c9f3cd196"
-          (reference "R13") (unit 1)
-        )
         (path "/0e4c4e8a-78e0-4f49-88dc-754c12656209/4037b4b4-0005-458e-a3e9-fe2ae826ab0c"
           (reference "R1") (unit 1)
@@
   (symbol (lib_id "Connector_Generic:Conn_01x06") (at 224.79 38.1 0) (unit 1)
     (in_bom yes) (on_board yes) (dnp no) (fields_autoplaced)
-    (property "Reference" "J4" (at 227.965 38.1 0)
+    (property "Reference" "J19" (at 227.965 38.1 0)
       (effects (font (size 1.27 1.27)) (justify left))
     )
@@
     (instances
       (project "fortuna-box"
-        (path "/0e4c4e8a-78e0-4f49-88dc-754c12656209"
-          (reference "J4") (unit 1)
-        )
-        (path "/0e4c4e8a-78e0-4f49-88dc-754c12656209/afd1b413-de30-4838-bb16-3d0c9f3cd196"
-          (reference "J7") (unit 1)
-        )
         (path "/0e4c4e8a-78e0-4f49-88dc-754c12656209/4037b4b4-0005-458e-a3e9-fe2ae826ab0c"
           (reference "J19") (unit 1)
@@
   (symbol (lib_id "Connector_Generic:Conn_01x10") (at 245.745 60.96 0) (mirror y) (unit 1)
     (in_bom yes) (on_board yes) (dnp no)
-    (property "Reference" "J2" (at 242.57 60.96 0)
+    (property "Reference" "J21" (at 242.57 60.96 0)
       (effects (font (size 1.27 1.27)) (justify left))
     )
@@
     (instances
       (project "fortuna-box"
-        (path "/0e4c4e8a-78e0-4f49-88dc-754c12656209"
-          (reference "J2") (unit 1)
-        )
         (path "/0e4c4e8a-78e0-4f49-88dc-754c12656209/4037b4b4-0005-458e-a3e9-fe2ae826ab0c"
           (reference "J21") (unit 1)
