File: circuit/cpu.kicad_sch (KiCad schematic)
At the start: 27 parts, among them J1 Port B, J2 Port C, J3 Port E, J4 Port A, J5 Port D, J6 Port F, U1 74HTC138

Commit message: .
Parts:
- removed JP1: Clock, symbol Jumper:Jumper_2_Open
- added J4: Port G, symbol Connector_Generic:Conn_02x03_Counter_Clockwise
- added Q1: 2N3904, Package_TO_SOT_THT:TO-92_Inline, symbol Transistor_BJT:2N3904
- added R?: 10k, symbol Device:R_US
- added R?: 1K, symbol Device:R_US
- added X?: 7.3728 MHz, Oscillator:Oscillator_DIP-14, symbol Oscillator:ACO-xxxMHz
- R?: value 1K -> 10k
Connections:
- net CLK: now also Q1.1 (E), R?.1
- net CLK_ENA: now also Q1.3 (C)
- net CLK_EXT: now also R?.2, X?.8 (OUT)
- net GND: now also R?.2, X?.7 (GND)
- net VCC: now also X?.14 (Vcc)
- net ~{RST}: now also C?.1, D?.2 (A), R?.1, R?.1
- new net: Q1.2 (B), R?.1
- new net RX: J4.6 (Pin_6)
- new net TX: J4.5 (Pin_5)
Other:
- note added: "CLOCK (opt 1)"
- note added: "CLOCK (opt 2)"
- note removed: "CLOCK"
- moved on the sheet: D2, R?, X?

Commit message: .
Parts:
- removed D2 (x2): 1N4148, Diode_THT:D_DO-35_SOD27_P7.62mm_Horizontal, symbol Diode:1N4148
- removed Q1: 2N3904, Package_TO_SOT_THT:TO-92_Inline, symbol Transistor_BJT:2N3904
- removed R? (x2): 10k, symbol Device:R_US
- removed R?: 1K, symbol Device:R_US
- removed X?: 7.3728 MHz, Oscillator:Oscillator_DIP-14, symbol Oscillator:ACO-xxxMHz
- added C2: 10uF, symbol Device:C
- added R?: 10K, symbol Device:R_US
- added U6: 74LS08, symbol 74xx:74LS08
Connections:
- net CLK: now also U6.3
- net CLK_ENA: now also R?.1, U6.1
- net CLK_EXT: now also U6.2
- net GND: now also C2.2
- net VCC: now also C2.1, R?.2
Other:
- note added: "CLOCK"
- note removed: "CLOCK (opt 1)"
- note removed: "CLOCK (opt 2)"
- moved on the sheet: X?

Commit message: .
Parts:
- removed J4: Port G, symbol Connector_Generic:Conn_02x03_Counter_Clockwise
- removed J4: Port A, symbol Connector_Generic:Conn_02x03_Counter_Clockwise
- added J4: Port A, symbol Connector_Generic:Conn_01x06
- added J43: Port G, symbol Connector_Generic:Conn_01x06
Connections:
- net A1: now also J4.6 (Pin_6)
- net A2: now also J4.5 (Pin_5)
- net A3: now also J4.4 (Pin_4)
- net GND: now also J4.2 (Pin_2)
- net RX: now also J43.1 (Pin_1)
- net TX: now also J43.2 (Pin_2)
- net VCC: now also J4.1 (Pin_1)
- net ~{RST}: now also J4.3 (Pin_3)

Commit message: .
Parts:
- removed J6: Port F, symbol Connector_Generic:Conn_01x10
- added J3: Port F, symbol Connector_Generic:Conn_01x08
Connections:
- net A16: now also J43.4 (Pin_4)
- net A17: now also J43.5 (Pin_5)
- net A18: now also J43.6 (Pin_6)
- net CLK: now also J3.7 (Pin_7)
- net CLK_ENA: now also J3.8 (Pin_8)
- net ~{BUSAK}: now also J3.3 (Pin_3)
- net ~{BUSRQ}: now also J3.2 (Pin_2)
- net ~{IORQ}: now also J3.6 (Pin_6)
- net ~{M1}: now also J3.5 (Pin_5)
- net ~{NMI}: now also J3.4 (Pin_4)
- net RAMONLY: now reaches J43.3 (Pin_3)
- no-connect marks 7 -> 8
Changed lines of the file:
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@@
   (junction (at 105.41 73.025) (diameter 0) (color 0 0 0 0)
   )
+  (no_connect (at 264.16 142.24))
   (no_connect (at 31.75 74.295))
   (no_connect (at 54.61 41.275))
@@
     (stroke (width 0) (type default))
   )
-  (wire (pts (xy 274.955 142.24) (xy 264.16 142.24))
-    (stroke (width 0) (type default))
-  )
   (wire (pts (xy 45.72 132.715) (xy 59.69 132.715))
     (stroke (width 0) (type default))
@@
     (stroke (width 0) (type default))
   )
-  (wire (pts (xy 274.955 139.7) (xy 264.16 139.7))
-    (stroke (width 0) (type default))
-  )
   (bus (pts (xy 162.56 60.325) (xy 162.56 57.785))
     (stroke (width 0) (type default))
   )
+  (wire (pts (xy 245.745 95.885) (xy 234.95 95.885))
+    (stroke (width 0) (type default))
+  )
   (wire (pts (xy 97.79 57.785) (xy 124.46 57.785))
     (stroke (width 0) (type default))
@@
     (stroke (width 0) (type default))
   )
+  (wire (pts (xy 234.95 90.805) (xy 245.745 90.805))
+    (stroke (width 0) (type default))
+  )
   (wire (pts (xy 193.04 127.635) (xy 203.835 127.635))
     (stroke (width 0) (type default))
@@
     (stroke (width 0) (type default))
   )
+  (wire (pts (xy 245.745 98.425) (xy 234.95 98.425))
+    (stroke (width 0) (type default))
+  )
   (wire (pts (xy 245.745 149.86) (xy 234.95 149.86))
     (stroke (width 0) (type default))
@@
     (stroke (width 0) (type default))
   )
+  (wire (pts (xy 245.745 93.345) (xy 234.95 93.345))
+    (stroke (width 0) (type default))
+  )
   (wire (pts (xy 245.745 144.78) (xy 234.95 144.78))
     (stroke (width 0) (type default))
@@
   )
   (wire (pts (xy 193.04 139.7) (xy 203.835 139.7))
-    (stroke (width 0) (type default))
-  )
-  (wire (pts (xy 274.955 137.16) (xy 264.16 137.16))
     (stroke (width 0) (type default))
   )
@@
     (effects (font (size 1.27 1.27)) (justify right bottom))
   )
-  (label "A17" (at 274.955 139.7 180) (fields_autoplaced)
-    (effects (font (size 1.27 1.27)) (justify right bottom))
-  )
   (label "Y3W" (at 193.04 120.015 0) (fields_autoplaced)
     (effects (font (size 1.27 1.27)) (justify left bottom))
@@
     (effects (font (size 1.27 1.27)) (justify right bottom))
   )
+  (label "A16" (at 245.745 93.345 180) (fields_autoplaced)
+    (effects (font (size 1.27 1.27)) (justify right bottom))
+  )
   (label "~{IORQ}" (at 87.63 93.345 0) (fields_autoplaced)
     (effects (font (size 1.27 1.27)) (justify left bottom))
@@
     (effects (font (size 1.27 1.27)) (justify left bottom))
   )
+  (label "A18" (at 245.745 98.425 180) (fields_autoplaced)
+    (effects (font (size 1.27 1.27)) (justify right bottom))
+  )
   (label "~{Y0R}" (at 246.38 45.72 180) (fields_autoplaced)
     (effects (font (size 1.27 1.27)) (justify right bottom))
@@
     (effects (font (size 1.27 1.27)) (justify right bottom))
   )
-  (label "A18" (at 274.955 142.24 180) (fields_autoplaced)
-    (effects (font (size 1.27 1.27)) (justify right bottom))
-  )
   (label "~{NMI}" (at 274.955 149.86 180) (fields_autoplaced)
     (effects (font (size 1.27 1.27)) (justify right bottom))
@@
     (effects (font (size 1.27 1.27)) (justify right bottom))
   )
+  (label "A17" (at 245.745 95.885 180) (fields_autoplaced)
+    (effects (font (size 1.27 1.27)) (justify right bottom))
+  )
   (label "~{BUSRQ}" (at 87.63 100.965 0) (fields_autoplaced)
     (effects (font (size 1.27 1.27)) (justify left bottom))
@@
     (effects (font (size 1.27 1.27)) (justify right bottom))
   )
-  (label "A16" (at 274.955 137.16 180) (fields_autoplaced)
-    (effects (font (size 1.27 1.27)) (justify right bottom))
-  )
   (label "A3" (at 193.04 93.345 0) (fields_autoplaced)
     (effects (font (size 1.27 1.27)) (justify left bottom))
@@
   )
   (label "D5" (at 245.745 117.475 180) (fields_autoplaced)
+    (effects (font (size 1.27 1.27)) (justify right bottom))
+  )
+  (label "RAMONLY" (at 245.745 90.805 180) (fields_autoplaced)
     (effects (font (size 1.27 1.27)) (justify right bottom))
   )
@@
     )
   )
-  (symbol (lib_id "Connector_Generic:Conn_01x10") (at 259.08 147.32 0) (mirror y) (unit 1)
-    (in_bom yes) (on_board yes) (dnp no)
-    (property "Reference" "J6" (at 255.905 147.32 0)
-      (effects (font (size 1.27 1.27)) (justify left))
-    )
-    (property "Value" "Port F" (at 255.905 149.86 0)
-      (effects (font (size 1.27 1.27)) (justify left))
-    )
-    (property "Footprint" "" (at 259.08 147.32 0)
-      (effects (font (size 1.27 1.27)) hide)
-    )
-    (property "Datasheet" "~" (at 259.08 147.32 0)
-      (effects (font (size 1.27 1.27)) hide)
-    )
-    (pin "1")
-    (pin "10")
-    (pin "2")
-    (pin "3")
-    (pin "4")
-    (pin "5")
-    (pin "6")
-    (pin "7")
-    (pin "8")
-    (pin "9")
-    (instances
-      (project "fortuna-box"
-        (path "/0e4c4e8a-78e0-4f49-88dc-754c12656209"
-          (reference "J6") (unit 1)
-        )
-        (path "/0e4c4e8a-78e0-4f49-88dc-754c12656209/afd1b413-de30-4838-bb16-3d0c9f3cd196"
-          (reference "J12") (unit 1)
-        )
-      )
-    )
-  )
   (symbol (lib_id "74xx:74LS138") (at 224.79 50.8 0) (unit 1)
     (in_bom yes) (on_board yes) (dnp no) (fields_autoplaced)
@@
         )
       )
+    )
+  )
+  (symbol (lib_id "Connector_Generic:Conn_01x08") (at 259.08 149.86 0) (mirror y) (unit 1)
+    (in_bom yes) (on_board yes) (dnp no)
+    (property "Reference" "J3" (at 256.54 149.86 0)
+      (effects (font (size 1.27 1.27)) (justify left))
+    )
+    (property "Value" "Port F" (at 256.54 152.4 0)
+      (effects (font (size 1.27 1.27)) (justify left))
+    )
+    (property "Footprint" "" (at 259.08 149.86 0)
+      (effects (font (size 1.27 1.27)) hide)
+    )
+    (property "Datasheet" "~" (at 259.08 149.86 0)
+      (effects (font (size 1.27 1.27)) hide)
+    )
+    (pin "1")
+    (pin "2")
+    (pin "3")
+    (pin "4")
+    (pin "5")
+    (pin "6")
+    (pin "7")
+    (pin "8")
+    (instances
+      (project "fortuna-box"
+        (path "/0e4c4e8a-78e0-4f49-88dc-754c12656209"
+          (reference "J3") (unit 1)
+        )
+        (path "/0e4c4e8a-78e0-4f49-88dc-754c12656209/afd1b413-de30-4838-bb16-3d0c9f3cd196"
+          (reference "J12") (unit 1)
+        )
+        (path "/0e4c4e8a-78e0-4f49-88dc-754c12656209/34f47b44-6e82-4397-9bc8-849df4113da9"
+          (reference "J13") (unit 1)
+        )
+      )

Commit message: .
Connections:
- net RAMONLY renamed ~{RAMONLY}
Changed lines of the file:
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@@
     (effects (font (size 1.27 1.27)) (justify left bottom))
+  )
+  (label "~{RAMONLY}" (at 245.745 90.805 180) (fields_autoplaced)
+    (effects (font (size 1.27 1.27)) (justify right bottom))
   )
   (label "~{M1}" (at 200.66 55.88 0) (fields_autoplaced)
@@
     (effects (font (size 1.27 1.27)) (justify right bottom))
   )
-  (label "RAMONLY" (at 245.745 90.805 180) (fields_autoplaced)
-    (effects (font (size 1.27 1.27)) (justify right bottom))
-  )

Commit message: .
Parts:
- removed D?: GREEN, symbol Device:LED
- removed P?: USB_C_Plug_USB2.0, symbol Connector:USB_C_Plug_USB2.0
- removed R?: 100, symbol Device:R_US
Connections:
- no-connect marks 8 -> 3
Other:
- note removed: "POWER"
- moved on the sheet: C?, D?, R?, SW?, U6A, U?, X?

Commit message: .
Parts:
- added J50: External button, symbol Connector_Generic:Conn_01x02
Connections:
- net GND: now also J50.2 (Pin_2)
- net at R?.2, SW?.2: now also J50.1 (Pin_1)
Other:
- note added: "74HC138 (mplex)"
- note added: "74HCT08 (and)"
- note added: "CLK"
- note added: "Z80"
- moved on the sheet: C?, D?, R?, SW?, U6A, U?, X?

Commit message: .
Parts:
- added R?: 10K, symbol Device:R_US
- added U8: 74LS125, symbol 74xx:74LS125
- added X?: 7.3728 MHz, Oscillator:Oscillator_DIP-14, symbol Oscillator:ACO-xxxMHz
Connections:
- net CLK: now also U8.3
- net CLK_ENA: now also R?.1, U8.1
- net CLK_EXT: now also U8.2, X?.8 (OUT)
- net GND: now also R?.2, X?.7 (GND)
- net VCC: now also X?.14 (Vcc)
Other:
- moved on the sheet: R?, U6A, X?
