File: circuit/cpu.kicad_sch (KiCad schematic)
At the start: 28 parts, among them J1 Port B, J2 Port C, J3 Port E, J3 Port F, J4 Port A, J43 Port G, J5 Port D, J50 External button, U1 74HTC138, U6 74LS08, U8 74LS125

Commit message: .
Parts:
- removed R?: 10K, symbol Device:R_US
- removed U6: 74LS08, symbol 74xx:74LS08
- removed X?: 7.3728 MHz, Oscillator:Oscillator_DIP-14, symbol Oscillator:ACO-xxxMHz
Other:
- moved on the sheet: R?, U8A, X?

Commit message: .
Connections:
- net ~{RAMONLY} is gone; now on net ~{IORQ}: J43.3 (Pin_3)
- net ~{IORQ}: no longer J3.6 (Pin_6)
- new net RAMONLY: J3.6 (Pin_6)
Changed lines of the file:
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@@
     (effects (font (size 1.27 1.27)) (justify left bottom))
   )
-  (label "~{RAMONLY}" (at 245.745 90.805 180) (fields_autoplaced)
+  (label "~{IORQ}" (at 245.745 90.805 180) (fields_autoplaced)
     (effects (font (size 1.27 1.27)) (justify right bottom))
   )
@@
     (effects (font (size 1.27 1.27)) (justify right bottom))
   )
-  (label "~{IORQ}" (at 274.955 154.94 180) (fields_autoplaced)
+  (label "RAMONLY" (at 274.955 154.94 180) (fields_autoplaced)
     (effects (font (size 1.27 1.27)) (justify right bottom))
   )

Commit message: .
Parts:
- removed C2: 10uF, symbol Device:C
- removed R?: 10K, symbol Device:R_US
- removed U8: 74LS125, symbol 74xx:74LS125
- added SW3: SW_SPDT, symbol Switch:SW_SPDT
Connections:
- net CLK: now also SW3.3 (C); no longer U?.6 (~{CLK})
- net CLK_EXT: now also SW3.1 (A)
- net CLK_ENA: no longer names the net of J3.8 (Pin_8)
- new net ZCLK: SW3.2 (B), U?.6 (~{CLK})
- no-connect marks 3 -> 4

Commit message: Redeployt
Parts:
- added R?: 10K, symbol Device:R_US
Connections:
- net VCC: now also R?.2
- net ~{IORQ}: now also R?.1
Other:
- moved on the sheet: R?

Commit message: .
Parts:
- renumbered J2 to J10, J3 to J11, J3 to J12, J43 to J33, J4 to J7, J1 to J8, J5 to J9
Changed lines of the file:
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@@
   (symbol (lib_id "Connector_Generic:Conn_01x10") (at 208.915 114.935 0) (unit 1)
     (in_bom yes) (on_board yes) (dnp no) (fields_autoplaced)
-    (property "Reference" "J1" (at 212.09 114.935 0)
+    (property "Reference" "J8" (at 212.09 114.935 0)
       (effects (font (size 1.27 1.27)) (justify left))
     )
@@
     (instances
       (project "fortuna-box"
-        (path "/0e4c4e8a-78e0-4f49-88dc-754c12656209"
-          (reference "J1") (unit 1)
-        )
         (path "/0e4c4e8a-78e0-4f49-88dc-754c12656209/afd1b413-de30-4838-bb16-3d0c9f3cd196"
           (reference "J8") (unit 1)
@@
   (symbol (lib_id "Connector_Generic:Conn_01x08") (at 208.915 144.78 0) (unit 1)
     (in_bom yes) (on_board yes) (dnp no) (fields_autoplaced)
-    (property "Reference" "J5" (at 212.09 144.78 0)
+    (property "Reference" "J9" (at 212.09 144.78 0)
       (effects (font (size 1.27 1.27)) (justify left))
     )
@@
     (instances
       (project "fortuna-box"
-        (path "/0e4c4e8a-78e0-4f49-88dc-754c12656209"
-          (reference "J5") (unit 1)
-        )
         (path "/0e4c4e8a-78e0-4f49-88dc-754c12656209/afd1b413-de30-4838-bb16-3d0c9f3cd196"
           (reference "J9") (unit 1)
@@
   (symbol (lib_id "Connector_Generic:Conn_01x06") (at 208.915 90.805 0) (unit 1)
     (in_bom yes) (on_board yes) (dnp no) (fields_autoplaced)
-    (property "Reference" "J4" (at 212.09 90.805 0)
+    (property "Reference" "J7" (at 212.09 90.805 0)
       (effects (font (size 1.27 1.27)) (justify left))
     )
@@
     (instances
       (project "fortuna-box"
-        (path "/0e4c4e8a-78e0-4f49-88dc-754c12656209"
-          (reference "J4") (unit 1)
-        )
         (path "/0e4c4e8a-78e0-4f49-88dc-754c12656209/afd1b413-de30-4838-bb16-3d0c9f3cd196"
           (reference "J7") (unit 1)
@@
   (symbol (lib_id "Connector_Generic:Conn_01x08") (at 229.87 144.78 0) (mirror y) (unit 1)
     (in_bom yes) (on_board yes) (dnp no)
-    (property "Reference" "J3" (at 227.33 144.78 0)
+    (property "Reference" "J11" (at 227.33 144.78 0)
       (effects (font (size 1.27 1.27)) (justify left))
     )
@@
     (instances
       (project "fortuna-box"
-        (path "/0e4c4e8a-78e0-4f49-88dc-754c12656209"
-          (reference "J3") (unit 1)
-        )
         (path "/0e4c4e8a-78e0-4f49-88dc-754c12656209/afd1b413-de30-4838-bb16-3d0c9f3cd196"
           (reference "J11") (unit 1)
@@
   (symbol (lib_id "Connector_Generic:Conn_01x10") (at 229.87 114.935 0) (mirror y) (unit 1)
     (in_bom yes) (on_board yes) (dnp no)
-    (property "Reference" "J2" (at 226.695 114.935 0)
+    (property "Reference" "J10" (at 226.695 114.935 0)
       (effects (font (size 1.27 1.27)) (justify left))
     )
@@
     (instances
       (project "fortuna-box"
-        (path "/0e4c4e8a-78e0-4f49-88dc-754c12656209"
-          (reference "J2") (unit 1)
-        )
         (path "/0e4c4e8a-78e0-4f49-88dc-754c12656209/afd1b413-de30-4838-bb16-3d0c9f3cd196"
           (reference "J10") (unit 1)
@@
   (symbol (lib_id "Connector_Generic:Conn_01x08") (at 259.08 149.86 0) (mirror y) (unit 1)
     (in_bom yes) (on_board yes) (dnp no)
-    (property "Reference" "J3" (at 256.54 149.86 0)
+    (property "Reference" "J12" (at 256.54 149.86 0)
       (effects (font (size 1.27 1.27)) (justify left))
     )
@@
     (instances
       (project "fortuna-box"
-        (path "/0e4c4e8a-78e0-4f49-88dc-754c12656209"
-          (reference "J3") (unit 1)
-        )
         (path "/0e4c4e8a-78e0-4f49-88dc-754c12656209/afd1b413-de30-4838-bb16-3d0c9f3cd196"
           (reference "J12") (unit 1)
         )
-        (path "/0e4c4e8a-78e0-4f49-88dc-754c12656209/34f47b44-6e82-4397-9bc8-849df4113da9"
-          (reference "J13") (unit 1)
-        )
       )
     )
@@
   (symbol (lib_id "Connector_Generic:Conn_01x06") (at 229.87 90.805 0) (mirror y) (unit 1)
     (in_bom yes) (on_board yes) (dnp no)
-    (property "Reference" "J43" (at 226.695 90.805 0)
+    (property "Reference" "J33" (at 226.695 90.805 0)
       (effects (font (size 1.27 1.27)) (justify left))
     )
@@
     (instances
       (project "fortuna-box"
-        (path "/0e4c4e8a-78e0-4f49-88dc-754c12656209"
-          (reference "J43") (unit 1)
-        )
         (path "/0e4c4e8a-78e0-4f49-88dc-754c12656209/afd1b413-de30-4838-bb16-3d0c9f3cd196"
           (reference "J33") (unit 1)
