File: circuit/debugger.kicad_sch (KiCad schematic)
At the start: 1 part

Commit message: .
Parts:
- added J1: Port B, symbol Connector_Generic:Conn_01x10
- added J2: Port C, symbol Connector_Generic:Conn_01x10
- added J3: Port E, symbol Connector_Generic:Conn_01x08
- added J32: To UART board, symbol Connector_Generic:Conn_01x02
- added J4: Port A, symbol Connector_Generic:Conn_02x03_Counter_Clockwise
- added J4: Port G, symbol Connector_Generic:Conn_02x03_Counter_Clockwise
- added J5: Port D, symbol Connector_Generic:Conn_01x08
- added J6: Port F, symbol Connector_Generic:Conn_01x10
- added SW1: SW_Push, symbol Switch:SW_Push
Connections:
- net A0: now also XA1.A0, J2.10 (Pin_10); no longer XA1.A11
- net A1: now also XA1.A1, J4.3 (Pin_3); no longer XA1.A9
- net A10: now also XA1.A10, J3.3 (Pin_3); no longer XA1.A8
- net A11: now also XA1.A11, J3.4 (Pin_4); no longer XA1.D10
- net A12: now also XA1.A12, J3.5 (Pin_5); no longer XA1.D11
- net A13: now also XA1.A13, J3.6 (Pin_6); no longer XA1.D9
- net A14: now also XA1.A14, J3.7 (Pin_7); no longer XA1.D7
- net A15: now also XA1.A15, J3.8 (Pin_8); no longer XA1.D5
- net A16: now also XA1.D10, J6.1 (Pin_1); no longer XA1.D24
- net A17: now also XA1.D11, J6.2 (Pin_2); no longer XA1.A15
- net A18: now also XA1.D12, J6.3 (Pin_3); no longer XA1.D39
- net A2: now also XA1.A2, J4.2 (Pin_2); no longer XA1.A7
- net A3: now also XA1.A3, J4.1 (Pin_1); no longer XA1.A5
- net A4: now also XA1.A4, J5.5 (Pin_5); no longer XA1.A3
- net A5: now also XA1.A5, J5.6 (Pin_6); no longer XA1.A1
- net A6: now also XA1.A6, J5.7 (Pin_7); no longer XA1.A0
- net A7: now also XA1.A7, J5.8 (Pin_8); no longer XA1.A2
- net A8: now also XA1.A8, J3.1 (Pin_1); no longer XA1.A4
- net A9: now also XA1.A9, J3.2 (Pin_2); no longer XA1.A6
- net CLK: now also XA1.D25, J6.9 (Pin_9); no longer XA1.D3 (D3_INT1)
- net D0: now also XA1.D37, J2.1 (Pin_1); no longer XA1.D16 (D16/TX2)
- net D1: now also XA1.D36, J2.2 (Pin_2); no longer XA1.D18 (D18/TX1)
- net D2: now also XA1.D35, J2.3 (Pin_3); no longer XA1.D12
- net D3: now also XA1.D34, J2.4 (Pin_4); no longer XA1.D4
- net D4: now also XA1.D33, J2.5 (Pin_5); no longer XA1.D2 (D2_INT0)
- net D5: now also XA1.D32, J2.6 (Pin_6); no longer XA1.D6
- net D6: now also XA1.D31, J2.7 (Pin_7); no longer XA1.D8
- net D7: now also XA1.D30, J2.8 (Pin_8); no longer XA1.D14 (D14/TX3)
- net GND: now also J4.5 (Pin_5), SW1.1
- net VCC: now also J4.6 (Pin_6)
- net ~{BUSAK}: now also XA1.D47, J6.5 (Pin_5); no longer XA1.D41
- net ~{BUSRQ}: now also XA1.D23, J6.4 (Pin_4); no longer XA1.D37
- net ~{INT}: now also XA1.D42, J2.9 (Pin_9); no longer XA1.D20 (D20/SDA)
- net ~{IORQ}: now also XA1.D48, J6.8 (Pin_8); no longer XA1.D28
- net ~{M1}: now also XA1.D49, J6.7 (Pin_7); no longer XA1.D33
- net ~{MREQ}: now also XA1.D29, J5.3 (Pin_3); no longer XA1.D26
- net ~{NMI}: now also XA1.D24, J6.6 (Pin_6); no longer XA1.D22
- net ~{RD}: now also XA1.D28, J5.2 (Pin_2); no longer XA1.D45
- net ~{ROM_WE}: now also XA1.D22, J5.4 (Pin_4); no longer XA1.D47
- net ~{RST}: now also J4.4 (Pin_4); no longer XA1.D35
- net ~{WR}: now also XA1.D27, J5.1 (Pin_1); no longer XA1.D43
- net at XA1.D17 (D17/RX2): now also J32.2 (Pin_2)
- net ~{WAIT}: now reaches XA1.D46
- net ~{WAIT}: now also J1.10 (Pin_10)
- net at XA1.RST1 (RESET): now also SW1.2
- new net: J32.1 (Pin_1), XA1.D16 (D16/TX2)
- new net CLK_ENA: J6.10 (Pin_10), XA1.D26
- new net CLK_EXT: J1.9 (Pin_9)
- new net RX: J4.6 (Pin_6)
- new net TX: J4.5 (Pin_5)
- new net Y0R: J1.2 (Pin_2)
- new net Y0W: J1.1 (Pin_1)
- new net Y1R: J1.4 (Pin_4)
- new net Y1W: J1.3 (Pin_3)
- new net Y2R: J1.6 (Pin_6)
- new net Y2W: J1.5 (Pin_5)
- new net Y3R: J1.8 (Pin_8)
- new net Y3W: J1.7 (Pin_7)
- no-connect marks 49 -> 26
Other:
- note added: "A6, A7"
- note added: "Connection Ports"
- note added: "DEBUGGER"
- note added: "PA"
- note added: "PB (read-only)"
- note added: "PC"
- note added: "PF"
- note added: "PK"
- note added: "PL (read-only)"
- note removed: "(pin 54)"
- note removed: "(pin 55)"
- note removed: "(pin 56)"
- note removed: "(pin 57)"
- note removed: "(pin 58)"
- note removed: "(pin 59)"
- note removed: "(pin 60)"
- note removed: "(pin 61)"
- note removed: "(pin 62)"
- note removed: "(pin 63)"
- note removed: "(pin 65)"
- note removed: "(pin 69)"
- moved on the sheet: XA1

Commit message: .
Parts:
- removed J32: To UART board, symbol Connector_Generic:Conn_01x02
- removed J4: Port A, symbol Connector_Generic:Conn_02x03_Counter_Clockwise
- removed J4: Port G, symbol Connector_Generic:Conn_02x03_Counter_Clockwise
- added J4: Port A, symbol Connector_Generic:Conn_01x06
- added J43: Port G, symbol Connector_Generic:Conn_01x06
Connections:
- net A1: now also J4.6 (Pin_6)
- net A2: now also J4.5 (Pin_5)
- net A3: now also J4.4 (Pin_4)
- net GND: now also J4.2 (Pin_2)
- net RX: now also XA1.D16 (D16/TX2), J43.1 (Pin_1)
- net TX: now also XA1.D17 (D17/RX2), J43.2 (Pin_2)
- net VCC: now also J4.1 (Pin_1)
- net ~{INT}: now also XA1.D44; no longer XA1.D42
- net ~{RST}: now also J4.3 (Pin_3)

Commit message: .
Parts:
- removed J6: Port F, symbol Connector_Generic:Conn_01x10
- added J3: Port F, symbol Connector_Generic:Conn_01x08
Connections:
- net A16: now also J43.4 (Pin_4)
- net A17: now also J43.5 (Pin_5)
- net A18: now also J43.6 (Pin_6)
- net CLK: now also J3.7 (Pin_7)
- net CLK_ENA: now also J3.8 (Pin_8)
- net ~{BUSAK}: now also J3.3 (Pin_3)
- net ~{BUSRQ}: now also J3.2 (Pin_2)
- net ~{IORQ}: now also J3.6 (Pin_6)
- net ~{M1}: now also J3.5 (Pin_5)
- net ~{NMI}: now also J3.4 (Pin_4)
- net RAMONLY: now reaches J43.3 (Pin_3)
- net RAMONLY: now also XA1.D21 (D21/SCL)

Commit message: .
Connections:
- net Y0W: now also XA1.D38
Other:
- note added: "PD7"
Changed lines of the file:
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@@
+    (stroke (width 0) (type default))
+  )
+  (wire (pts (xy 123.825 121.92) (xy 134.62 121.92))
     (stroke (width 0) (type default))
   )
@@
     (effects (font (size 1.27 1.27) italic) (justify right bottom))
   )
+  (text "PD7" (at 138.43 121.92 0)
+    (effects (font (size 1.27 1.27)) (justify left bottom))
+  )
   (text "PL\n(read-only)" (at 139.065 140.97 0)
     (effects (font (size 1.27 1.27)) (justify left bottom))
@@
     (effects (font (size 1.27 1.27)) (justify left bottom))
   )
+  (label "Y0W" (at 134.62 121.92 180) (fields_autoplaced)
+    (effects (font (size 1.27 1.27)) (justify right bottom))
+  )
   (label "A6" (at 186.69 89.535 0) (fields_autoplaced)

Commit message: .
Connections:
- net Y0W: now also XA1.D15 (D15/RX3); no longer XA1.D38
- no-connect marks 26 -> 25
Other:
- note added: "PJ0"
- note removed: "PD7"
Changed lines of the file:
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@@
   (no_connect (at 57.785 124.46))
   (no_connect (at 57.785 50.8))
-  (no_connect (at 57.785 66.04))
   (no_connect (at 57.785 160.02))
   (no_connect (at 57.785 157.48))
@@
     (stroke (width 0) (type default))
   )
-  (wire (pts (xy 123.825 121.92) (xy 134.62 121.92))
-    (stroke (width 0) (type default))
-  )
   (wire (pts (xy 53.975 164.465) (xy 53.975 149.86))
     (stroke (width 0) (type default))
@@
   )
   (wire (pts (xy 46.99 121.92) (xy 57.785 121.92))
+    (stroke (width 0) (type default))
+  )
+  (wire (pts (xy 57.785 66.04) (xy 46.99 66.04))
     (stroke (width 0) (type default))
   )
@@
     (effects (font (size 1.27 1.27) italic) (justify right bottom))
   )
-  (text "PD7" (at 138.43 121.92 0)
-    (effects (font (size 1.27 1.27)) (justify left bottom))
-  )
   (text "PL\n(read-only)" (at 139.065 140.97 0)
     (effects (font (size 1.27 1.27)) (justify left bottom))
@@
     (effects (font (size 1.27 1.27)) (justify left bottom))
   )
+  (text "PJ0" (at 43.18 66.04 0)
+    (effects (font (size 1.27 1.27)) (justify right bottom))
+  )
   (text "PC" (at 138.43 111.76 0)
     (effects (font (size 1.27 1.27)) (justify left bottom))
@@
     (effects (font (size 1.27 1.27)) (justify right bottom))
   )
+  (label "Y0W" (at 46.99 66.04 0) (fields_autoplaced)
+    (effects (font (size 1.27 1.27)) (justify left bottom))
+  )
   (label "A11" (at 46.99 111.76 0) (fields_autoplaced)
     (effects (font (size 1.27 1.27)) (justify left bottom))
@@
     (effects (font (size 1.27 1.27)) (justify left bottom))
   )
-  (label "Y0W" (at 134.62 121.92 180) (fields_autoplaced)
-    (effects (font (size 1.27 1.27)) (justify right bottom))
-  )
   (label "A6" (at 186.69 89.535 0) (fields_autoplaced)

Commit message: .
Connections:
- net ~{RST}: now also XA1.D14 (D14/TX3)
- no-connect marks 25 -> 24
Other:
- note added: "PJ1"
Changed lines of the file:
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@@
   (no_connect (at 57.785 160.02))
   (no_connect (at 57.785 157.48))
-  (no_connect (at 57.785 68.58))
   (no_connect (at 57.785 147.32))
   (no_connect (at 57.785 58.42))
@@
     (stroke (width 0) (type default))
   )
+  (wire (pts (xy 46.99 68.58) (xy 57.785 68.58))
+    (stroke (width 0) (type default))
+  )
   (wire (pts (xy 46.99 99.06) (xy 57.785 99.06))
     (stroke (width 0) (type default))
@@
     (effects (font (size 1.27 1.27) italic) (justify right bottom))
   )
+  (text "PJ1" (at 43.18 68.58 0)
+    (effects (font (size 1.27 1.27)) (justify right bottom))
+  )
   (text "PL\n(read-only)" (at 139.065 140.97 0)
     (effects (font (size 1.27 1.27)) (justify left bottom))
@@
     (effects (font (size 1.27 1.27)) (justify left bottom))
   )
+  (label "~{RST}" (at 46.99 68.58 0) (fields_autoplaced)
+    (effects (font (size 1.27 1.27)) (justify left bottom))
+  )

Commit message: .
Connections:
- net RAMONLY renamed ~{RAMONLY}
Changed lines of the file:
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@@
     (effects (font (size 1.27 1.27)) (justify left bottom))
-  )
-  (label "RAMONLY" (at 239.395 28.575 180) (fields_autoplaced)
-    (effects (font (size 1.27 1.27)) (justify right bottom))
   )
   (label "D4" (at 134.62 109.22 180) (fields_autoplaced)
@@
     (effects (font (size 1.27 1.27)) (justify right bottom))
   )
+  (label "~{RAMONLY}" (at 239.395 28.575 180) (fields_autoplaced)
+    (effects (font (size 1.27 1.27)) (justify right bottom))
+  )
   (label "CLK" (at 268.605 94.615 180) (fields_autoplaced)
     (effects (font (size 1.27 1.27)) (justify right bottom))
@@
     (effects (font (size 1.27 1.27)) (justify right bottom))
   )
+  (label "~{RAMONLY}" (at 46.99 73.66 0) (fields_autoplaced)
+    (effects (font (size 1.27 1.27)) (justify left bottom))
+  )
   (label "Y3R" (at 186.69 59.69 0) (fields_autoplaced)
     (effects (font (size 1.27 1.27)) (justify left bottom))
@@
     (effects (font (size 1.27 1.27)) (justify left bottom))
   )
-  (label "RAMONLY" (at 46.99 73.66 0) (fields_autoplaced)
-    (effects (font (size 1.27 1.27)) (justify left bottom))
-  )

Commit message: .
Connections:
- net ~{IORQ}: now also J43.3 (Pin_3); no longer J3.6 (Pin_6)
- net ~{RAMONLY}: no longer J43.3 (Pin_3)
- new net RAMONLY: J3.6 (Pin_6)
Changed lines of the file:
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@@
     (effects (font (size 1.27 1.27)) (justify left bottom))
   )
-  (label "~{IORQ}" (at 268.605 92.075 180) (fields_autoplaced)
+  (label "RAMONLY" (at 268.605 92.075 180) (fields_autoplaced)
     (effects (font (size 1.27 1.27)) (justify right bottom))
   )
@@
     (effects (font (size 1.27 1.27)) (justify right bottom))
   )
-  (label "~{RAMONLY}" (at 239.395 28.575 180) (fields_autoplaced)
+  (label "~{IORQ}" (at 239.395 28.575 180) (fields_autoplaced)
     (effects (font (size 1.27 1.27)) (justify right bottom))
   )
