File: circuit/debugger.kicad_sch (KiCad schematic)
At the start: 9 parts, among them J1 Port B, J2 Port C, J3 Port E, J3 Port F, J4 Port A, J43 Port G, J5 Port D, SW1 SW_Push

Commit message: .
Connections:
- net CLK_ENA: no longer names the net of J3.8 (Pin_8)
- net CLK_ENA: no longer XA1.D26
- no-connect marks 24 -> 25
Other:
- moved on the sheet: J3
Changed lines of the file:
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@@
   (no_connect (at 94.615 39.37))
   (no_connect (at 92.075 39.37))
-  (no_connect (at 257.81 79.375))
+  (no_connect (at 257.81 78.74))
   (no_connect (at 57.785 137.16))
+  (no_connect (at 257.81 96.52))
   (no_connect (at 86.995 39.37))
   (no_connect (at 57.785 142.24))
@@
     (stroke (width 0) (type default))
   )
-  (wire (pts (xy 134.62 91.44) (xy 123.825 91.44))
-    (stroke (width 0) (type default))
-  )
   (wire (pts (xy 186.69 31.115) (xy 197.485 31.115))
     (stroke (width 0) (type default))
@@
     (stroke (width 0) (type default))
   )
-  (wire (pts (xy 268.605 92.075) (xy 257.81 92.075))
+  (wire (pts (xy 268.605 91.44) (xy 257.81 91.44))
     (stroke (width 0) (type default))
   )
@@
     (stroke (width 0) (type default))
   )
-  (wire (pts (xy 268.605 81.915) (xy 257.81 81.915))
+  (wire (pts (xy 268.605 81.28) (xy 257.81 81.28))
     (stroke (width 0) (type default))
   )
@@
     (stroke (width 0) (type default))
   )
-  (wire (pts (xy 268.605 89.535) (xy 257.81 89.535))
+  (wire (pts (xy 268.605 88.9) (xy 257.81 88.9))
     (stroke (width 0) (type default))
   )
@@
     (stroke (width 0) (type default))
   )
-  (wire (pts (xy 268.605 97.155) (xy 257.81 97.155))
-    (stroke (width 0) (type default))
-  )
   (wire (pts (xy 239.395 57.15) (xy 228.6 57.15))
     (stroke (width 0) (type default))
@@
     (stroke (width 0) (type default))
   )
-  (wire (pts (xy 268.605 86.995) (xy 257.81 86.995))
+  (wire (pts (xy 268.605 86.36) (xy 257.81 86.36))
     (stroke (width 0) (type default))
   )
@@
     (stroke (width 0) (type default))
   )
-  (wire (pts (xy 268.605 94.615) (xy 257.81 94.615))
+  (wire (pts (xy 268.605 93.98) (xy 257.81 93.98))
     (stroke (width 0) (type default))
   )
@@
     (stroke (width 0) (type default))
   )
-  (wire (pts (xy 268.605 84.455) (xy 257.81 84.455))
+  (wire (pts (xy 268.605 83.82) (xy 257.81 83.82))
     (stroke (width 0) (type default))
   )
@@
     (effects (font (size 1.27 1.27)) (justify left bottom))
   )
-  (label "RAMONLY" (at 268.605 92.075 180) (fields_autoplaced)
+  (label "RAMONLY" (at 268.605 91.44 180) (fields_autoplaced)
     (effects (font (size 1.27 1.27)) (justify right bottom))
   )
@@
     (effects (font (size 1.27 1.27)) (justify right bottom))
   )
-  (label "CLK" (at 268.605 94.615 180) (fields_autoplaced)
+  (label "CLK" (at 268.605 93.98 180) (fields_autoplaced)
     (effects (font (size 1.27 1.27)) (justify right bottom))
   )
@@
     (effects (font (size 1.27 1.27)) (justify left bottom))
   )
-  (label "~{NMI}" (at 268.605 86.995 180) (fields_autoplaced)
+  (label "~{NMI}" (at 268.605 86.36 180) (fields_autoplaced)
     (effects (font (size 1.27 1.27)) (justify right bottom))
   )
@@
     (effects (font (size 1.27 1.27)) (justify right bottom))
   )
-  (label "CLK_ENA" (at 268.605 97.155 180) (fields_autoplaced)
-    (effects (font (size 1.27 1.27)) (justify right bottom))
-  )
   (label "GND" (at 186.69 26.035 0) (fields_autoplaced)
     (effects (font (size 1.27 1.27)) (justify left bottom))
@@
     (effects (font (size 1.27 1.27)) (justify left bottom))
   )
-  (label "~{M1}" (at 268.605 89.535 180) (fields_autoplaced)
+  (label "~{M1}" (at 268.605 88.9 180) (fields_autoplaced)
     (effects (font (size 1.27 1.27)) (justify right bottom))
   )
@@
     (effects (font (size 1.27 1.27)) (justify left bottom))
   )
-  (label "~{BUSAK}" (at 268.605 84.455 180) (fields_autoplaced)
-    (effects (font (size 1.27 1.27)) (justify right bottom))
-  )
-  (label "~{BUSRQ}" (at 268.605 81.915 180) (fields_autoplaced)
+  (label "~{BUSAK}" (at 268.605 83.82 180) (fields_autoplaced)
+    (effects (font (size 1.27 1.27)) (justify right bottom))
+  )
+  (label "~{BUSRQ}" (at 268.605 81.28 180) (fields_autoplaced)
     (effects (font (size 1.27 1.27)) (justify right bottom))
   )
@@
     (effects (font (size 1.27 1.27)) (justify left bottom))
   )
-  (label "CLK_ENA" (at 134.62 91.44 180) (fields_autoplaced)
-    (effects (font (size 1.27 1.27)) (justify right bottom))
-  )
   (label "~{RST}" (at 186.69 28.575 0) (fields_autoplaced)
     (effects (font (size 1.27 1.27)) (justify left bottom))
@@
     (effects (font (size 1.27 1.27)) (justify left bottom))
   )
-  (symbol (lib_id "Connector_Generic:Conn_01x08") (at 252.73 86.995 0) (mirror y) (unit 1)
+  (symbol (lib_id "Connector_Generic:Conn_01x08") (at 252.73 86.36 0) (mirror y) (unit 1)
     (in_bom yes) (on_board yes) (dnp no)
-    (property "Reference" "J3" (at 250.19 86.995 0)
+    (property "Reference" "J3" (at 250.19 86.36 0)
       (effects (font (size 1.27 1.27)) (justify left))
     )
-    (property "Value" "Port F" (at 250.19 89.535 0)
+    (property "Value" "Port F" (at 250.19 88.9 0)
       (effects (font (size 1.27 1.27)) (justify left))
     )
-    (property "Footprint" "" (at 252.73 86.995 0)
+    (property "Footprint" "" (at 252.73 86.36 0)
       (effects (font (size 1.27 1.27)) hide)
     )
-    (property "Datasheet" "~" (at 252.73 86.995 0)
+    (property "Datasheet" "~" (at 252.73 86.36 0)
       (effects (font (size 1.27 1.27)) hide)
     )

Commit message: .
Parts:
- renumbered J3 to J13, J4 to J26, J1 to J27, J5 to J28, J2 to J29, J3 to J30, J43 to J38
Changed lines of the file:
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@@
   (symbol (lib_id "Connector_Generic:Conn_01x08") (at 252.73 86.36 0) (mirror y) (unit 1)
     (in_bom yes) (on_board yes) (dnp no)
-    (property "Reference" "J3" (at 250.19 86.36 0)
+    (property "Reference" "J13" (at 250.19 86.36 0)
       (effects (font (size 1.27 1.27)) (justify left))
     )
@@
     (instances
       (project "fortuna-box"
-        (path "/0e4c4e8a-78e0-4f49-88dc-754c12656209"
-          (reference "J3") (unit 1)
-        )
-        (path "/0e4c4e8a-78e0-4f49-88dc-754c12656209/afd1b413-de30-4838-bb16-3d0c9f3cd196"
-          (reference "J11") (unit 1)
-        )
         (path "/0e4c4e8a-78e0-4f49-88dc-754c12656209/34f47b44-6e82-4397-9bc8-849df4113da9"
           (reference "J13") (unit 1)
@@
   (symbol (lib_id "Connector_Generic:Conn_01x06") (at 202.565 28.575 0) (unit 1)
     (in_bom yes) (on_board yes) (dnp no) (fields_autoplaced)
-    (property "Reference" "J4" (at 205.74 28.575 0)
+    (property "Reference" "J26" (at 205.74 28.575 0)
       (effects (font (size 1.27 1.27)) (justify left))
     )
@@
     (instances
       (project "fortuna-box"
-        (path "/0e4c4e8a-78e0-4f49-88dc-754c12656209"
-          (reference "J4") (unit 1)
-        )
-        (path "/0e4c4e8a-78e0-4f49-88dc-754c12656209/afd1b413-de30-4838-bb16-3d0c9f3cd196"
-          (reference "J7") (unit 1)
-        )
         (path "/0e4c4e8a-78e0-4f49-88dc-754c12656209/34f47b44-6e82-4397-9bc8-849df4113da9"
           (reference "J26") (unit 1)
@@
   (symbol (lib_id "Connector_Generic:Conn_01x06") (at 223.52 28.575 0) (mirror y) (unit 1)
     (in_bom yes) (on_board yes) (dnp no)
-    (property "Reference" "J43" (at 220.345 28.575 0)
+    (property "Reference" "J38" (at 220.345 28.575 0)
       (effects (font (size 1.27 1.27)) (justify left))
     )
@@
     (instances
       (project "fortuna-box"
-        (path "/0e4c4e8a-78e0-4f49-88dc-754c12656209"
-          (reference "J43") (unit 1)
-        )
-        (path "/0e4c4e8a-78e0-4f49-88dc-754c12656209/afd1b413-de30-4838-bb16-3d0c9f3cd196"
-          (reference "J33") (unit 1)
-        )
         (path "/0e4c4e8a-78e0-4f49-88dc-754c12656209/34f47b44-6e82-4397-9bc8-849df4113da9"
           (reference "J38") (unit 1)
@@
   (symbol (lib_id "Connector_Generic:Conn_01x08") (at 223.52 81.915 0) (mirror y) (unit 1)
     (in_bom yes) (on_board yes) (dnp no)
-    (property "Reference" "J3" (at 220.98 81.915 0)
+    (property "Reference" "J30" (at 220.98 81.915 0)
       (effects (font (size 1.27 1.27)) (justify left))
     )
@@
     (instances
       (project "fortuna-box"
-        (path "/0e4c4e8a-78e0-4f49-88dc-754c12656209"
-          (reference "J3") (unit 1)
-        )
-        (path "/0e4c4e8a-78e0-4f49-88dc-754c12656209/afd1b413-de30-4838-bb16-3d0c9f3cd196"
-          (reference "J11") (unit 1)
-        )
         (path "/0e4c4e8a-78e0-4f49-88dc-754c12656209/34f47b44-6e82-4397-9bc8-849df4113da9"
           (reference "J30") (unit 1)
@@
   (symbol (lib_id "Connector_Generic:Conn_01x08") (at 202.565 81.915 0) (unit 1)
     (in_bom yes) (on_board yes) (dnp no) (fields_autoplaced)
-    (property "Reference" "J5" (at 205.74 81.915 0)
+    (property "Reference" "J28" (at 205.74 81.915 0)
       (effects (font (size 1.27 1.27)) (justify left))
     )
@@
     (instances
       (project "fortuna-box"
-        (path "/0e4c4e8a-78e0-4f49-88dc-754c12656209"
-          (reference "J5") (unit 1)
-        )
-        (path "/0e4c4e8a-78e0-4f49-88dc-754c12656209/afd1b413-de30-4838-bb16-3d0c9f3cd196"
-          (reference "J9") (unit 1)
-        )
         (path "/0e4c4e8a-78e0-4f49-88dc-754c12656209/34f47b44-6e82-4397-9bc8-849df4113da9"
           (reference "J28") (unit 1)
@@
   (symbol (lib_id "Connector_Generic:Conn_01x10") (at 223.52 52.07 0) (mirror y) (unit 1)
     (in_bom yes) (on_board yes) (dnp no)
-    (property "Reference" "J2" (at 220.345 52.07 0)
+    (property "Reference" "J29" (at 220.345 52.07 0)
       (effects (font (size 1.27 1.27)) (justify left))
     )
@@
     (instances
       (project "fortuna-box"
-        (path "/0e4c4e8a-78e0-4f49-88dc-754c12656209"
-          (reference "J2") (unit 1)
-        )
-        (path "/0e4c4e8a-78e0-4f49-88dc-754c12656209/afd1b413-de30-4838-bb16-3d0c9f3cd196"
-          (reference "J10") (unit 1)
-        )
         (path "/0e4c4e8a-78e0-4f49-88dc-754c12656209/34f47b44-6e82-4397-9bc8-849df4113da9"
           (reference "J29") (unit 1)
@@
   (symbol (lib_id "Connector_Generic:Conn_01x10") (at 202.565 52.07 0) (unit 1)
     (in_bom yes) (on_board yes) (dnp no) (fields_autoplaced)
-    (property "Reference" "J1" (at 205.74 52.07 0)
+    (property "Reference" "J27" (at 205.74 52.07 0)
       (effects (font (size 1.27 1.27)) (justify left))
     )
@@
     (instances
       (project "fortuna-box"
-        (path "/0e4c4e8a-78e0-4f49-88dc-754c12656209"
-          (reference "J1") (unit 1)
-        )
-        (path "/0e4c4e8a-78e0-4f49-88dc-754c12656209/afd1b413-de30-4838-bb16-3d0c9f3cd196"
-          (reference "J8") (unit 1)
-        )
         (path "/0e4c4e8a-78e0-4f49-88dc-754c12656209/34f47b44-6e82-4397-9bc8-849df4113da9"
           (reference "J27") (unit 1)
