File: circuit/power.kicad_sch (KiCad schematic)
At the start: 10 parts, among them J1 Port B, J2 Port C, J3 Port E, J3 Port F, J4 Port A, J43 Port G, J5 Port D

Commit message: .
Connections:
- net ~{RAMONLY} is gone; now on net ~{IORQ}: J43.3 (Pin_3)
- net ~{IORQ}: no longer J3.6 (Pin_6)
- new net RAMONLY: J3.6 (Pin_6)
Changed lines of the file:
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@@
     (effects (font (size 3 3) (thickness 0.6) bold) (justify left bottom))
   )
-  (label "~{RAMONLY}" (at 192.405 50.8 180) (fields_autoplaced)
+  (label "~{IORQ}" (at 192.405 50.8 180) (fields_autoplaced)
     (effects (font (size 1.27 1.27)) (justify right bottom))
   )
@@
     (effects (font (size 1.27 1.27)) (justify right bottom))
   )
-  (label "~{IORQ}" (at 221.615 114.935 180) (fields_autoplaced)
+  (label "RAMONLY" (at 221.615 114.935 180) (fields_autoplaced)
     (effects (font (size 1.27 1.27)) (justify right bottom))
   )
