File: circuit/storage.kicad_sch (KiCad schematic)
At the start: 24 parts, among them J1 Port B, J15 TX (debug), J16 ISCP header, J2 Port C, J3 SDCard, J4 Port A, J43 Port G, U11 ATtiny2313-20P, U19 4013, U8 74HC595, Y1 16Mhz

Commit message: .
Parts:
- removed J15: TX (debug), symbol Connector_Generic:Conn_01x01
- added R18: 10k, symbol Device:R_US
Connections:
- net SD_MISO: now also R18.2
- net VCC: now also R18.1

Commit message: .
Parts:
- removed R14, R15: 10k, symbol Device:R_US
- removed U11: ATtiny2313-20P, Package_DIP:DIP-20_W7.62mm, symbol MCU_Microchip_ATtiny:ATtiny2313-20P
- removed U8: 74HC595, symbol 74xx:74HC595
- added D4: D, symbol Device:D
- added U3: ATmega328-P, Package_DIP:DIP-28_W7.62mm, symbol MCU_Microchip_ATmega:ATmega328-P
- added U9: 74LS374, symbol 74xx:74LS374
- renumbered D1 to D5, J4 to J17, J1 to J23, J2 to J24, J43 to J36
Connections:
- net SD_MISO is gone; now on net MISO: J3.4 (Pin_4), R18.2
- net D0: now also U3.2 (PD0), U9.2 (O0), U9.3 (D0)
- net D1: now also U3.3 (PD1), U9.4 (D1), U9.5 (O1)
- net D2: now also U3.4 (PD2), U9.6 (O2), U9.7 (D2)
- net D3: now also U3.5 (PD3), U9.8 (D3), U9.9 (O3)
- net D4: now also U3.6 (PD4), U9.12 (O4), U9.13 (D4)
- net D5: now also U3.11 (PD5), U9.14 (D5), U9.15 (O5)
- net D6: now also U3.12 (PD6), U9.16 (O6), U9.17 (D6)
- net D7: now also U3.13 (PD7), U9.18 (D7), U9.19 (O7)
- net GND: now also U3.22 (GND), U3.8 (GND), U9.10 (GND); no longer R13.2
- net MISO: now also U3.18 (PB4); no longer J16.5 (Pin_5), J3.3 (Pin_3)
- net MOSI: now also J3.3 (Pin_3), U3.17 (PB3)
- net R: now also U3.24 (PC1); no longer R13.1
- net RST: now also R13.2, U3.1 (~{RESET}/PC6)
- net SCK: now also U3.19 (PB5)
- net VCC: now also R13.1, U3.7 (VCC), U9.20 (VCC)
- net Y2R: now also U3.14 (PB0), U9.1 (OE)
- net Y2W: now also U3.25 (PC2)
- net ~{WAIT}: now also D4.1 (K); no longer U19.2 (~{Q})
- net at C12.1, Y1.2: now also U3.9 (XTAL1/PB6)
- net at U19.1 (Q): no longer D5.2 (A)
- net at C18.1, Y1.1: now also U3.10 (XTAL2/PB7)
- new net: D4.2 (A), U19.2 (~{Q})
- new net FF_CLK: U3.26 (PC3), U9.11 (Cp)
- new net LED: D5.2 (A), U3.23 (PC0)
- new net SD_MOSI: J16.5 (Pin_5)
- no-connect marks 1 -> 2
Other:
- note added: "74HC374"
- note added: "ATMEGA328"
- note removed: "74HC595"
- note removed: "ATTINY2313"
- moved on the sheet: C12, C18, D5, J16, J3, R12, R18, R?, U19A, U?D, Y1

Commit message: .
Parts:
- removed J16: ISCP header, symbol Connector_Generic:Conn_01x06
- added J16: Fortuna programmer, symbol Connector_Generic:Conn_01x08
- added Q2: 2N3904, Package_TO_SOT_THT:TO-92_Inline, symbol Transistor_BJT:2N3904
- added R14: 10k, symbol Device:R_US
- Y1: value 16Mhz -> 16.5 Mhz
Connections:
- net D1: now also R14.1
- net FF_CLK: now also U3.25 (PC2); no longer U3.26 (PC3)
- net GND: now also J16.1 (Pin_1), Q2.1 (E)
- net MISO: now also J16.4 (Pin_4)
- net RST: now also J16.6 (Pin_6)
- net RX: now also J16.7 (Pin_7)
- net SCK: now also J16.2 (Pin_2)
- net SD_MOSI: now also J16.5 (Pin_5)
- net VCC: now also J16.3 (Pin_3)
- net Y2W: now also U3.15 (PB1); no longer U3.25 (PC2)
- new net DEBUG: Q2.2 (B)
- new net TX_DEBUG: Q2.3 (C), R14.2

Commit message: .
Parts:
- removed C2: 10uF, symbol Device:C
- removed Q2: 2N3904, Package_TO_SOT_THT:TO-92_Inline, symbol Transistor_BJT:2N3904
- removed R14: 10k, symbol Device:R_US
- removed U9: 74LS374, symbol 74xx:74LS374
- added D6, D7: D, symbol Device:D
Connections:
- net Y2R: now also D7.2 (A)
- net Y2W: now also D6.2 (A); no longer U?.9
- net FF_CLK: no longer names the net of U3.25 (PC2)
- new net: D6.1 (K), D7.1 (K), U?.9
- no-connect marks 2 -> 7
Other:
- moved on the sheet: D4, U19A, U?D

Commit message: .
Parts:
- added U8: 74HCT04, symbol 74xx:74HCT04
Connections:
- net Y2R: now also U8.3; no longer D7.2 (A)
- net Y2W: now also U?.9; no longer D6.2 (A)
- net at U19.6 (S): now also D6.1 (K), D7.1 (K); no longer U?.8
- new net: D7.2 (A), U8.4
- new net: D6.2 (A), U?.8
Other:
- moved on the sheet: D6, D7, U?D
Changed lines of the file:
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@@
   (junction (at 142.24 59.69) (diameter 0) (color 0 0 0 0)
   )
+  (junction (at 35.56 53.34) (diameter 0) (color 0 0 0 0)
+  )
   (junction (at 53.34 125.73) (diameter 0) (color 0 0 0 0)
   )
@@
   (junction (at 132.08 59.69) (diameter 0) (color 0 0 0 0)
   )
-  (junction (at 35.56 40.64) (diameter 0) (color 0 0 0 0)
-  )
-  (junction (at 33.02 22.86) (diameter 0) (color 0 0 0 0)
-  )
-  (junction (at 38.1 25.4) (diameter 0) (color 0 0 0 0)
+  (junction (at 31.75 22.86) (diameter 0) (color 0 0 0 0)
+  )
+  (junction (at 40.64 25.4) (diameter 0) (color 0 0 0 0)
   )
   (no_connect (at 167.64 67.31))
@@
     (stroke (width 0) (type default))
   )
-  (wire (pts (xy 38.1 38.1) (xy 38.1 40.64))
-    (stroke (width 0) (type default))
-  )
   (wire (pts (xy 218.44 67.945) (xy 229.235 67.945))
     (stroke (width 0) (type default))
@@
     (stroke (width 0) (type default))
   )
-  (wire (pts (xy 38.1 25.4) (xy 76.2 25.4))
+  (wire (pts (xy 16.51 25.4) (xy 40.64 25.4))
     (stroke (width 0) (type default))
   )
@@
     (stroke (width 0) (type default))
   )
-  (wire (pts (xy 16.51 25.4) (xy 38.1 25.4))
-    (stroke (width 0) (type default))
-  )
   (wire (pts (xy 142.24 59.69) (xy 139.7 59.69))
     (stroke (width 0) (type default))
@@
     (stroke (width 0) (type default))
   )
-  (wire (pts (xy 33.02 38.1) (xy 33.02 40.64))
-    (stroke (width 0) (type default))
-  )
   (wire (pts (xy 256.54 34.29) (xy 256.54 43.18))
     (stroke (width 0) (type default))
@@
     (stroke (width 0) (type default))
   )
-  (wire (pts (xy 35.56 58.42) (xy 35.56 62.23))
+  (wire (pts (xy 35.56 53.34) (xy 35.56 62.23))
     (stroke (width 0) (type default))
   )
@@
     (stroke (width 0) (type default))
   )
+  (wire (pts (xy 40.64 25.4) (xy 76.2 25.4))
+    (stroke (width 0) (type default))
+  )
   (wire (pts (xy 147.32 57.15) (xy 147.32 59.69))
     (stroke (width 0) (type default))
@@
     (stroke (width 0) (type default))
   )
-  (wire (pts (xy 16.51 22.86) (xy 33.02 22.86))
+  (wire (pts (xy 16.51 22.86) (xy 31.75 22.86))
     (stroke (width 0) (type default))
   )
@@
     (stroke (width 0) (type default))
   )
-  (wire (pts (xy 38.1 40.64) (xy 35.56 40.64))
-    (stroke (width 0) (type default))
-  )
   (wire (pts (xy 218.44 96.52) (xy 229.235 96.52))
     (stroke (width 0) (type default))
@@
     (stroke (width 0) (type default))
   )
-  (wire (pts (xy 33.02 22.86) (xy 76.2 22.86))
-    (stroke (width 0) (type default))
-  )
-  (wire (pts (xy 33.02 22.86) (xy 33.02 30.48))
+  (wire (pts (xy 31.75 22.86) (xy 76.2 22.86))
+    (stroke (width 0) (type default))
+  )
+  (wire (pts (xy 31.75 22.86) (xy 31.75 30.48))
     (stroke (width 0) (type default))
   )
@@
     (stroke (width 0) (type default))
   )
+  (wire (pts (xy 35.56 53.34) (xy 40.64 53.34))
+    (stroke (width 0) (type default))
+  )
   (wire (pts (xy 218.44 65.405) (xy 229.235 65.405))
     (stroke (width 0) (type default))
@@
     (stroke (width 0) (type default))
   )
-  (wire (pts (xy 33.02 40.64) (xy 35.56 40.64))
-    (stroke (width 0) (type default))
-  )
   (wire (pts (xy 271.145 75.565) (xy 260.35 75.565))
     (stroke (width 0) (type default))
@@
     (stroke (width 0) (type default))
   )
+  (wire (pts (xy 31.75 53.34) (xy 35.56 53.34))
+    (stroke (width 0) (type default))
+  )
   (wire (pts (xy 156.21 49.53) (xy 167.64 49.53))
     (stroke (width 0) (type default))
@@
     (stroke (width 0) (type default))
   )
-  (wire (pts (xy 38.1 25.4) (xy 38.1 30.48))
-    (stroke (width 0) (type default))
-  )
   (wire (pts (xy 55.88 138.43) (xy 55.88 140.97))
     (stroke (width 0) (type default))
@@
     (stroke (width 0) (type default))
   )
-  (wire (pts (xy 35.56 40.64) (xy 35.56 43.18))
+  (wire (pts (xy 40.64 25.4) (xy 40.64 30.48))
     (stroke (width 0) (type default))
   )
@@
     )
   )
-  (symbol (lib_id "Device:D") (at 38.1 34.29 90) (unit 1)
-    (in_bom yes) (on_board yes) (dnp no) (fields_autoplaced)
-    (property "Reference" "D7" (at 40.64 33.02 90)
+  (symbol (lib_id "Device:D") (at 40.64 49.53 90) (unit 1)
+    (in_bom yes) (on_board yes) (dnp no) (fields_autoplaced)
+    (property "Reference" "D7" (at 43.18 48.26 90)
       (effects (font (size 1.27 1.27)) (justify right))
     )
-    (property "Value" "D" (at 40.64 35.56 90)
+    (property "Value" "D" (at 43.18 50.8 90)
       (effects (font (size 1.27 1.27)) (justify right))
     )
-    (property "Footprint" "" (at 38.1 34.29 0)
-      (effects (font (size 1.27 1.27)) hide)
-    )
-    (property "Datasheet" "~" (at 38.1 34.29 0)
-      (effects (font (size 1.27 1.27)) hide)
-    )
-    (property "Sim.Device" "D" (at 38.1 34.29 0)
-      (effects (font (size 1.27 1.27)) hide)
-    )
-    (property "Sim.Pins" "1=K 2=A" (at 38.1 34.29 0)
+    (property "Footprint" "" (at 40.64 49.53 0)
+      (effects (font (size 1.27 1.27)) hide)
+    )
+    (property "Datasheet" "~" (at 40.64 49.53 0)
+      (effects (font (size 1.27 1.27)) hide)
+    )
+    (property "Sim.Device" "D" (at 40.64 49.53 0)
+      (effects (font (size 1.27 1.27)) hide)
+    )
+    (property "Sim.Pins" "1=K 2=A" (at 40.64 49.53 0)
       (effects (font (size 1.27 1.27)) hide)
     )
@@
     )
   )
-  (symbol (lib_id "Device:D") (at 33.02 34.29 90) (unit 1)
+  (symbol (lib_id "Device:D") (at 31.75 49.53 90) (unit 1)
     (in_bom yes) (on_board yes) (dnp no)
-    (property "Reference" "D6" (at 27.94 33.02 90)
+    (property "Reference" "D6" (at 26.67 48.26 90)
       (effects (font (size 1.27 1.27)) (justify right))
     )
-    (property "Value" "D" (at 29.21 35.56 90)
+    (property "Value" "D" (at 27.94 50.8 90)
       (effects (font (size 1.27 1.27)) (justify right))
     )
-    (property "Footprint" "" (at 33.02 34.29 0)
-      (effects (font (size 1.27 1.27)) hide)
-    )
-    (property "Datasheet" "~" (at 33.02 34.29 0)
-      (effects (font (size 1.27 1.27)) hide)
-    )
-    (property "Sim.Device" "D" (at 33.02 34.29 0)
-      (effects (font (size 1.27 1.27)) hide)
-    )
-    (property "Sim.Pins" "1=K 2=A" (at 33.02 34.29 0)
+    (property "Footprint" "" (at 31.75 49.53 0)
+      (effects (font (size 1.27 1.27)) hide)
+    )
+    (property "Datasheet" "~" (at 31.75 49.53 0)
+      (effects (font (size 1.27 1.27)) hide)
+    )
+    (property "Sim.Device" "D" (at 31.75 49.53 0)
+      (effects (font (size 1.27 1.27)) hide)
+    )
+    (property "Sim.Pins" "1=K 2=A" (at 31.75 49.53 0)
       (effects (font (size 1.27 1.27)) hide)
     )
@@
     )
   )
-  (symbol (lib_id "74xx:74HCT04") (at 35.56 50.8 270) (unit 4)
+  (symbol (lib_id "74xx:74HCT04") (at 40.64 38.1 270) (unit 2)
     (in_bom yes) (on_board yes) (dnp no)
-    (property "Reference" "U?" (at 39.37 53.34 0)
-      (effects (font (size 1.27 1.27)))
-    )
-    (property "Value" "74HCT04" (at 41.91 50.8 0)
-      (effects (font (size 1.27 1.27)))
-    )
-    (property "Footprint" "" (at 35.56 50.8 0)
-      (effects (font (size 1.27 1.27)) hide)
-    )
-    (property "Datasheet" "https://assets.nexperia.com/documents/data-sheet/74HC_HCT04.pdf" (at 35.56 50.8 0)
-      (effects (font (size 1.27 1.27)) hide)
-    )
+    (property "Reference" "U8" (at 44.45 39.37 0)
+      (effects (font (size 1.27 1.27)))
+    )
+    (property "Value" "74HCT04" (at 46.99 38.1 0)
+      (effects (font (size 1.27 1.27)))
+    )
+    (property "Footprint" "" (at 40.64 38.1 0)
+      (effects (font (size 1.27 1.27)) hide)
+    )
+    (property "Datasheet" "https://assets.nexperia.com/documents/data-sheet/74HC_HCT04.pdf" (at 40.64 38.1 0)
+      (effects (font (size 1.27 1.27)) hide)
+    )
+    (pin "1")
+    (pin "2")
+    (pin "3")
+    (pin "4")
+    (pin "5")
+    (pin "6")
+    (pin "8")
+    (pin "9")
+    (pin "10")
+    (pin "11")
+    (pin "12")
+    (pin "13")
+    (pin "14")
+    (pin "7")
+    (instances
+      (project "fortuna-box"
+        (path "/0e4c4e8a-78e0-4f49-88dc-754c12656209/0ad0c907-f2a9-47ff-aff1-7aaecbdef7ee"
+          (reference "U8") (unit 2)
+        )
+      )
+    )
+  )
+  (symbol (lib_id "74xx:74HCT04") (at 31.75 38.1 270) (unit 4)
+    (in_bom yes) (on_board yes) (dnp no)
+    (property "Reference" "U?" (at 26.67 39.37 0)
+      (effects (font (size 1.27 1.27)))
+    )
+    (property "Value" "74HCT04" (at 24.13 38.1 0)
+      (effects (font (size 1.27 1.27)))
+    )
+    (property "Footprint" "" (at 31.75 38.1 0)
+      (effects (font (size 1.27 1.27)) hide)
+    )
+    (property "Datasheet" "https://assets.nexperia.com/documents/data-sheet/74HC_HCT04.pdf" (at 31.75 38.1 0)
+      (effects (font (size 1.27 1.27)) hide)
+    )

Commit message: .
Connections:
- net D0: now also U3.25 (PC2); no longer U3.2 (PD0)
- net D1: now also U3.26 (PC3); no longer U3.3 (PD1)
- net D2: now also U3.27 (PC4); no longer U3.4 (PD2)
- net D3: now also U3.28 (PC5); no longer U3.5 (PD3)
- net RX: now also U3.3 (PD1)
- net TX: now also J16.8 (Pin_8), U3.2 (PD0)
- net Y2R: now also U3.4 (PD2); no longer U3.14 (PB0)
- net Y2W: now also U3.5 (PD3); no longer U3.15 (PB1)
- no-connect marks 7 -> 5
Changed lines of the file:
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@@
   (junction (at 40.64 25.4) (diameter 0) (color 0 0 0 0)
   )
-  (no_connect (at 167.64 67.31))
   (no_connect (at 167.64 44.45))
-  (no_connect (at 167.64 72.39))
-  (no_connect (at 167.64 74.93))
+  (no_connect (at 167.64 39.37))
   (no_connect (at 198.12 39.37))
-  (no_connect (at 167.64 69.85))
+  (no_connect (at 167.64 41.91))
   (no_connect (at 43.18 67.31))
   (wire (pts (xy 218.44 75.565) (xy 229.235 75.565))
@@
     (stroke (width 0) (type default))
   )
+  (wire (pts (xy 156.21 69.85) (xy 167.64 69.85))
+    (stroke (width 0) (type default))
+  )
   (wire (pts (xy 142.24 52.07) (xy 139.7 52.07))
     (stroke (width 0) (type default))
@@
     (stroke (width 0) (type default))
   )
-  (wire (pts (xy 91.44 95.25) (xy 167.64 95.25))
+  (wire (pts (xy 156.21 95.25) (xy 167.64 95.25))
     (stroke (width 0) (type default))
   )
@@
     (stroke (width 0) (type default))
   )
-  (wire (pts (xy 91.44 97.79) (xy 167.64 97.79))
+  (wire (pts (xy 156.21 97.79) (xy 167.64 97.79))
     (stroke (width 0) (type default))
   )
@@
     (stroke (width 0) (type default))
   )
-  (wire (pts (xy 167.64 39.37) (xy 156.21 39.37))
-    (stroke (width 0) (type default))
-  )
   (wire (pts (xy 35.56 81.28) (xy 77.47 81.28))
     (stroke (width 0) (type default))
   )
+  (wire (pts (xy 156.21 74.93) (xy 167.64 74.93))
+    (stroke (width 0) (type default))
+  )
   (wire (pts (xy 24.13 69.85) (xy 27.94 69.85))
     (stroke (width 0) (type default))
@@
     (stroke (width 0) (type default))
   )
-  (wire (pts (xy 91.44 85.09) (xy 167.64 85.09))
+  (wire (pts (xy 233.68 26.67) (xy 233.68 34.29))
     (stroke (width 0) (type default))
   )
@@
     (stroke (width 0) (type default))
   )
+  (wire (pts (xy 156.21 85.09) (xy 167.64 85.09))
+    (stroke (width 0) (type default))
+  )
   (wire (pts (xy 132.08 59.69) (xy 132.08 62.23))
     (stroke (width 0) (type default))
   )
-  (wire (pts (xy 91.44 82.55) (xy 167.64 82.55))
-    (stroke (width 0) (type default))
-  )
   (wire (pts (xy 31.75 22.86) (xy 76.2 22.86))
     (stroke (width 0) (type default))
@@
     (stroke (width 0) (type default))
   )
-  (wire (pts (xy 167.64 41.91) (xy 156.21 41.91))
+  (wire (pts (xy 156.21 72.39) (xy 167.64 72.39))
+    (stroke (width 0) (type default))
+  )
+  (wire (pts (xy 167.64 87.63) (xy 156.21 87.63))
     (stroke (width 0) (type default))
   )
@@
     (stroke (width 0) (type default))
   )
-  (wire (pts (xy 91.44 100.33) (xy 167.64 100.33))
+  (wire (pts (xy 156.21 100.33) (xy 167.64 100.33))
     (stroke (width 0) (type default))
   )
@@
     (stroke (width 0) (type default))
   )
-  (wire (pts (xy 91.44 92.71) (xy 167.64 92.71))
+  (wire (pts (xy 156.21 82.55) (xy 167.64 82.55))
+    (stroke (width 0) (type default))
+  )
+  (wire (pts (xy 156.21 92.71) (xy 167.64 92.71))
     (stroke (width 0) (type default))
   )
@@
     (stroke (width 0) (type default))
   )
+  (wire (pts (xy 156.21 67.31) (xy 167.64 67.31))
+    (stroke (width 0) (type default))
+  )
   (wire (pts (xy 182.88 27.94) (xy 182.88 31.75))
     (stroke (width 0) (type default))
@@
     (stroke (width 0) (type default))
   )
-  (wire (pts (xy 91.44 90.17) (xy 167.64 90.17))
-    (stroke (width 0) (type default))
-  )
   (wire (pts (xy 19.05 85.09) (xy 29.21 85.09))
     (stroke (width 0) (type default))
@@
     (stroke (width 0) (type default))
   )
-  (wire (pts (xy 91.44 87.63) (xy 167.64 87.63))
+  (wire (pts (xy 167.64 90.17) (xy 156.21 90.17))
     (stroke (width 0) (type default))
   )
@@
     (effects (font (size 1.27 1.27)) (justify left bottom))
   )
+  (label "RX" (at 156.21 85.09 0) (fields_autoplaced)
+    (effects (font (size 1.27 1.27)) (justify left bottom))
+  )
   (label "Y2W" (at 16.51 22.86 0) (fields_autoplaced)
     (effects (font (size 1.27 1.27)) (justify left bottom))
@@
     (effects (font (size 1.27 1.27)) (justify left bottom))
   )
+  (label "TX" (at 233.68 26.67 270) (fields_autoplaced)
+    (effects (font (size 1.27 1.27)) (justify right bottom))
+  )
   (label "Y2W" (at 218.44 91.44 0) (fields_autoplaced)
     (effects (font (size 1.27 1.27)) (justify left bottom))
@@
     (effects (font (size 1.27 1.27)) (justify right bottom))
   )
-  (label "Y2W" (at 156.21 41.91 0) (fields_autoplaced)
-    (effects (font (size 1.27 1.27)) (justify left bottom))
-  )
   (label "SCK" (at 26.67 128.27 0) (fields_autoplaced)
     (effects (font (size 1.27 1.27)) (justify left bottom))
@@
     (effects (font (size 1.27 1.27)) (justify left bottom))
   )
-  (label "D4" (at 91.44 92.71 0) (fields_autoplaced)
+  (label "D4" (at 156.21 92.71 0) (fields_autoplaced)
     (effects (font (size 1.27 1.27)) (justify left bottom))
   )
@@
     (effects (font (size 1.27 1.27)) (justify left bottom))
   )
-  (label "D5" (at 91.44 95.25 0) (fields_autoplaced)
-    (effects (font (size 1.27 1.27)) (justify left bottom))
-  )
-  (label "D0" (at 91.44 82.55 0) (fields_autoplaced)
+  (label "D5" (at 156.21 95.25 0) (fields_autoplaced)
     (effects (font (size 1.27 1.27)) (justify left bottom))
   )
@@
     (effects (font (size 1.27 1.27)) (justify left bottom))
   )
-  (label "D2" (at 91.44 87.63 0) (fields_autoplaced)
-    (effects (font (size 1.27 1.27)) (justify left bottom))
-  )
   (label "D3" (at 271.145 88.9 180) (fields_autoplaced)
     (effects (font (size 1.27 1.27)) (justify right bottom))
   )
+  (label "D0" (at 156.21 67.31 0) (fields_autoplaced)
+    (effects (font (size 1.27 1.27)) (justify left bottom))
+  )
   (label "RX" (at 236.22 26.67 270) (fields_autoplaced)
     (effects (font (size 1.27 1.27)) (justify right bottom))
@@
     (effects (font (size 1.27 1.27)) (justify right bottom))
   )
-  (label "D1" (at 91.44 85.09 0) (fields_autoplaced)
-    (effects (font (size 1.27 1.27)) (justify left bottom))
-  )
   (label "LED" (at 156.21 62.23 0) (fields_autoplaced)
     (effects (font (size 1.27 1.27)) (justify left bottom))
@@
     (effects (font (size 1.27 1.27)) (justify right bottom))
   )
-  (label "D7" (at 91.44 100.33 0) (fields_autoplaced)
+  (label "D7" (at 156.21 100.33 0) (fields_autoplaced)
     (effects (font (size 1.27 1.27)) (justify left bottom))
   )
@@
     (effects (font (size 1.27 1.27)) (justify left bottom))
   )
+  (label "D3" (at 156.21 74.93 0) (fields_autoplaced)
+    (effects (font (size 1.27 1.27)) (justify left bottom))
+  )
+  (label "TX" (at 156.21 82.55 0) (fields_autoplaced)
+    (effects (font (size 1.27 1.27)) (justify left bottom))
+  )
+  (label "D2" (at 156.21 72.39 0) (fields_autoplaced)
+    (effects (font (size 1.27 1.27)) (justify left bottom))
+  )
   (label "TX" (at 271.145 65.405 180) (fields_autoplaced)
     (effects (font (size 1.27 1.27)) (justify right bottom))
@@
     (effects (font (size 1.27 1.27)) (justify right bottom))
   )
+  (label "Y2R" (at 156.21 87.63 0) (fields_autoplaced)
+    (effects (font (size 1.27 1.27)) (justify left bottom))
+  )
+  (label "D1" (at 156.21 69.85 0) (fields_autoplaced)
+    (effects (font (size 1.27 1.27)) (justify left bottom))
+  )
   (label "~{IORQ}" (at 271.145 67.945 180) (fields_autoplaced)
     (effects (font (size 1.27 1.27)) (justify right bottom))
@@
     (effects (font (size 1.27 1.27)) (justify left bottom))
   )
-  (label "Y2R" (at 156.21 39.37 0) (fields_autoplaced)
-    (effects (font (size 1.27 1.27)) (justify left bottom))
-  )
   (label "LED" (at 179.07 128.27 0) (fields_autoplaced)
     (effects (font (size 1.27 1.27)) (justify left bottom))
@@
     (effects (font (size 1.27 1.27)) (justify left bottom))
   )
-  (label "D6" (at 91.44 97.79 0) (fields_autoplaced)
+  (label "D6" (at 156.21 97.79 0) (fields_autoplaced)
     (effects (font (size 1.27 1.27)) (justify left bottom))
   )
@@
     (effects (font (size 1.27 1.27)) (justify left bottom))
   )
-  (label "D3" (at 91.44 90.17 0) (fields_autoplaced)
-    (effects (font (size 1.27 1.27)) (justify left bottom))
-  )
+  (label "Y2W" (at 156.21 90.17 0) (fields_autoplaced)
+    (effects (font (size 1.27 1.27)) (justify left bottom))
+  )

Commit message: .
Parts:
- removed D6, D7: D, symbol Device:D
- removed U8: 74HCT04, symbol 74xx:74HCT04
- added U8: 74HCT595, symbol 74xx:74HCT595
Connections:
- net D0: now also U8.15 (QA)
- net D1: now also U8.1 (QB)
- net D2: now also U8.2 (QC)
- net D3: now also U8.3 (QD)
- net D4: now also U8.4 (QE)
- net D5: now also U8.5 (QF)
- net D6: now also U8.6 (QG)
- net D7: now also U8.7 (QH)
- net GND: now also U8.8 (GND)
- net MOSI: now also U8.14 (SER)
- net SCK: now also U8.11 (SRCLK)
- net SD_CS: now also U3.15 (PB1)
- net VCC: now also U8.10 (~{SRCLR}), U8.16 (VCC)
- net Y2R: now also U8.13 (~{OE})
- net RCLK: now reaches U3.14 (PB0)
- net RCLK: now also U8.12 (RCLK)
- net at U19.6 (S): now also U?.8
- no-connect marks 5 -> 4
Other:
- moved on the sheet: D4, D5, R?, U19A, U?D

Commit message: .
Parts:
- J3: value SDCard -> Adafruit SDCard Module
Other:
- moved on the sheet: J3, R12, R18
