File: circuit/storage.kicad_sch (KiCad schematic)
At the start: 22 parts, among them J16 Fortuna programmer, J17 Port A, J23 Port B, J24 Port C, J3 Adafruit SDCard Module, J36 Port G, U19 4013, U3 ATmega328-P, U8 74HCT595, Y1 16.5 Mhz

Commit message: .
Parts:
- added R14, R15: 10k, symbol Device:R_US
Connections:
- net RX: now also R15.2
- net SD_CS: now also U3.16 (PB2); no longer U3.15 (PB1)
- net TX: now also R14.2
- net VCC: now also R14.1, R15.1
Changed lines of the file:
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@@
   (junction (at 132.08 59.69) (diameter 0) (color 0 0 0 0)
   )
+  (junction (at 111.76 60.96) (diameter 0) (color 0 0 0 0)
+  )
+  (junction (at 120.65 85.09) (diameter 0) (color 0 0 0 0)
+  )
   (junction (at 35.56 22.86) (diameter 0) (color 0 0 0 0)
   )
+  (junction (at 111.76 82.55) (diameter 0) (color 0 0 0 0)
+  )
   (junction (at 106.68 107.95) (diameter 0) (color 0 0 0 0)
   )
-  (no_connect (at 167.64 44.45))
+  (junction (at 102.87 60.96) (diameter 0) (color 0 0 0 0)
+  )
   (no_connect (at 198.12 39.37))
   (no_connect (at 129.54 139.7))
+  (no_connect (at 167.64 41.91))
   (no_connect (at 43.18 59.69))
   (wire (pts (xy 218.44 75.565) (xy 229.235 75.565))
     (stroke (width 0) (type default))
   )
+  (wire (pts (xy 120.65 71.12) (xy 120.65 85.09))
+    (stroke (width 0) (type default))
+  )
   (wire (pts (xy 218.44 67.945) (xy 229.235 67.945))
     (stroke (width 0) (type default))
@@
     (stroke (width 0) (type default))
   )
+  (wire (pts (xy 111.76 60.96) (xy 120.65 60.96))
+    (stroke (width 0) (type default))
+  )
   (wire (pts (xy 142.24 52.07) (xy 139.7 52.07))
     (stroke (width 0) (type default))
@@
     (stroke (width 0) (type default))
   )
+  (wire (pts (xy 120.65 85.09) (xy 167.64 85.09))
+    (stroke (width 0) (type default))
+  )
   (wire (pts (xy 271.145 99.06) (xy 260.35 99.06))
     (stroke (width 0) (type default))
@@
     (stroke (width 0) (type default))
   )
+  (wire (pts (xy 102.87 55.88) (xy 102.87 60.96))
+    (stroke (width 0) (type default))
+  )
   (wire (pts (xy 156.21 97.79) (xy 167.64 97.79))
     (stroke (width 0) (type default))
@@
     (stroke (width 0) (type default))
   )
-  (wire (pts (xy 156.21 41.91) (xy 167.64 41.91))
-    (stroke (width 0) (type default))
-  )
   (wire (pts (xy 46.99 123.19) (xy 46.99 133.35))
     (stroke (width 0) (type default))
@@
     (stroke (width 0) (type default))
   )
+  (wire (pts (xy 111.76 60.96) (xy 111.76 63.5))
+    (stroke (width 0) (type default))
+  )
   (wire (pts (xy 45.72 64.77) (xy 45.72 77.47))
     (stroke (width 0) (type default))
@@
     (stroke (width 0) (type default))
   )
+  (wire (pts (xy 156.21 44.45) (xy 167.64 44.45))
+    (stroke (width 0) (type default))
+  )
   (wire (pts (xy 142.24 59.69) (xy 147.32 59.69))
     (stroke (width 0) (type default))
   )
+  (wire (pts (xy 111.76 82.55) (xy 167.64 82.55))
+    (stroke (width 0) (type default))
+  )
   (wire (pts (xy 218.44 96.52) (xy 229.235 96.52))
     (stroke (width 0) (type default))
@@
     (stroke (width 0) (type default))
   )
-  (wire (pts (xy 156.21 85.09) (xy 167.64 85.09))
+  (wire (pts (xy 91.44 85.09) (xy 120.65 85.09))
     (stroke (width 0) (type default))
   )
@@
     (stroke (width 0) (type default))
   )
+  (wire (pts (xy 102.87 60.96) (xy 102.87 63.5))
+    (stroke (width 0) (type default))
+  )
   (wire (pts (xy 218.44 99.06) (xy 229.235 99.06))
     (stroke (width 0) (type default))
@@
     (stroke (width 0) (type default))
   )
+  (wire (pts (xy 120.65 60.96) (xy 120.65 63.5))
+    (stroke (width 0) (type default))
+  )
   (wire (pts (xy 167.64 64.77) (xy 156.21 64.77))
     (stroke (width 0) (type default))
@@
     (stroke (width 0) (type default))
   )
-  (wire (pts (xy 156.21 82.55) (xy 167.64 82.55))
+  (wire (pts (xy 91.44 82.55) (xy 111.76 82.55))
     (stroke (width 0) (type default))
   )
@@
     (stroke (width 0) (type default))
   )
+  (wire (pts (xy 102.87 60.96) (xy 111.76 60.96))
+    (stroke (width 0) (type default))
+  )
   (wire (pts (xy 140.97 132.08) (xy 129.54 132.08))
     (stroke (width 0) (type default))
@@
   )
   (wire (pts (xy 140.97 134.62) (xy 129.54 134.62))
+    (stroke (width 0) (type default))
+  )
+  (wire (pts (xy 111.76 71.12) (xy 111.76 82.55))
     (stroke (width 0) (type default))
   )
@@
     (effects (font (size 1.27 1.27)) (justify left bottom))
   )
-  (label "RX" (at 156.21 85.09 0) (fields_autoplaced)
+  (label "RX" (at 91.44 85.09 0) (fields_autoplaced)
     (effects (font (size 1.27 1.27)) (justify left bottom))
   )
@@
     (effects (font (size 1.27 1.27)) (justify left bottom))
   )
-  (label "SD_CS" (at 156.21 41.91 0) (fields_autoplaced)
-    (effects (font (size 1.27 1.27)) (justify left bottom))
-  )
   (label "A1" (at 218.44 75.565 0) (fields_autoplaced)
     (effects (font (size 1.27 1.27)) (justify left bottom))
@@
     (effects (font (size 1.27 1.27)) (justify left bottom))
   )
-  (label "TX" (at 156.21 82.55 0) (fields_autoplaced)
+  (label "TX" (at 91.44 82.55 0) (fields_autoplaced)
     (effects (font (size 1.27 1.27)) (justify left bottom))
   )
@@
   (label "D5" (at 140.97 129.54 180) (fields_autoplaced)
     (effects (font (size 1.27 1.27)) (justify right bottom))
+  )
+  (label "SD_CS" (at 156.21 44.45 0) (fields_autoplaced)
+    (effects (font (size 1.27 1.27)) (justify left bottom))
   )
   (label "D7" (at 271.145 99.06 180) (fields_autoplaced)
@@
         (path "/0e4c4e8a-78e0-4f49-88dc-754c12656209/0ad0c907-f2a9-47ff-aff1-7aaecbdef7ee"
           (reference "C8") (unit 1)
+        )
+      )
+    )
+  )
+  (symbol (lib_id "Device:R_US") (at 120.65 67.31 0) (mirror y) (unit 1)
+    (in_bom yes) (on_board yes) (dnp no) (fields_autoplaced)
+    (property "Reference" "R15" (at 118.11 66.04 0)
+      (effects (font (size 1.27 1.27)) (justify left))
+    )
+    (property "Value" "10k" (at 118.11 68.58 0)
+      (effects (font (size 1.27 1.27)) (justify left))
+    )
+    (property "Footprint" "" (at 119.634 67.564 90)
+      (effects (font (size 1.27 1.27)) hide)
+    )
+    (property "Datasheet" "~" (at 120.65 67.31 0)
+      (effects (font (size 1.27 1.27)) hide)
+    )
+    (pin "1")
+    (pin "2")
+    (instances
+      (project "fortuna-box"
+        (path "/0e4c4e8a-78e0-4f49-88dc-754c12656209/0ad0c907-f2a9-47ff-aff1-7aaecbdef7ee"
+          (reference "R15") (unit 1)
         )
       )
@@
     )
   )
+  (symbol (lib_id "Device:R_US") (at 111.76 67.31 0) (mirror y) (unit 1)
+    (in_bom yes) (on_board yes) (dnp no) (fields_autoplaced)
+    (property "Reference" "R14" (at 109.22 66.04 0)
+      (effects (font (size 1.27 1.27)) (justify left))
+    )
+    (property "Value" "10k" (at 109.22 68.58 0)
+      (effects (font (size 1.27 1.27)) (justify left))
+    )
+    (property "Footprint" "" (at 110.744 67.564 90)
+      (effects (font (size 1.27 1.27)) hide)
+    )
+    (property "Datasheet" "~" (at 111.76 67.31 0)
+      (effects (font (size 1.27 1.27)) hide)
+    )
+    (pin "1")
+    (pin "2")
+    (instances
+      (project "fortuna-box"
+        (path "/0e4c4e8a-78e0-4f49-88dc-754c12656209/0ad0c907-f2a9-47ff-aff1-7aaecbdef7ee"
+          (reference "R14") (unit 1)
+        )
+      )
+    )
+  )
   (symbol (lib_id "power:VCC") (at 46.99 115.57 0) (unit 1)
     (in_bom yes) (on_board yes) (dnp no) (fields_autoplaced)
@@
     )
   )
-  (symbol (lib_id "power:VCC") (at 102.87 63.5 0) (mirror y) (unit 1)
-    (in_bom yes) (on_board yes) (dnp no) (fields_autoplaced)
-    (property "Reference" "#PWR012" (at 102.87 67.31 0)
-      (effects (font (size 1.27 1.27)) hide)
-    )
-    (property "Value" "VCC" (at 102.87 58.42 0)
-      (effects (font (size 1.27 1.27)))
-    )
-    (property "Footprint" "" (at 102.87 63.5 0)
-      (effects (font (size 1.27 1.27)) hide)
-    )
-    (property "Datasheet" "" (at 102.87 63.5 0)
-      (effects (font (size 1.27 1.27)) hide)
-    )
+  (symbol (lib_id "power:VCC") (at 102.87 55.88 0) (mirror y) (unit 1)
+    (in_bom yes) (on_board yes) (dnp no) (fields_autoplaced)
+    (property "Reference" "#PWR012" (at 102.87 59.69 0)
+      (effects (font (size 1.27 1.27)) hide)
+    )
+    (property "Value" "VCC" (at 102.87 50.8 0)
+      (effects (font (size 1.27 1.27)))
+    )
+    (property "Footprint" "" (at 102.87 55.88 0)
+      (effects (font (size 1.27 1.27)) hide)
+    )
+    (property "Datasheet" "" (at 102.87 55.88 0)
+      (effects (font (size 1.27 1.27)) hide)
+    )

Commit message: .
Parts:
- removed C12, C18: 22pF, symbol Device:C
- removed D4: D, symbol Device:D
- removed D5: LED BLUE, symbol Device:LED
- removed R13, R14, R15: 10k, symbol Device:R_US
- removed R?: 2K, symbol Device:R_US
- removed U19: 4013, symbol 4xxx:4013
- removed U3: ATmega328-P, Package_DIP:DIP-28_W7.62mm, symbol MCU_Microchip_ATmega:ATmega328-P
- removed U8: 74HCT595, symbol 74xx:74HCT595
- removed U?: 74HCT04, symbol 74xx:74HCT04
- removed Y1: 16.5 Mhz, symbol Device:Crystal
- added D4: LED, symbol Device:LED
- added Q1: 2N3906, Package_TO_SOT_THT:TO-92_Inline, symbol Transistor_BJT:2N3906
- added R13: 10k, symbol Device:R
- added R14: 220, symbol Device:R
- added U9: Pico, RPi_Pico:RPi_Pico_SMD_TH, symbol MCU_RaspberryPi_and_Boards:Pico
Connections:
- net GND: now also D4.1 (K), U9.21 (GPIO16)
- net MISO: now also U9.1 (GPIO0)
- net MOSI: now also U9.5 (GPIO3)
- net SCK: now also U9.4 (GPIO2)
- net SD_CS: now also R13.1, U9.2 (GPIO1)
- net VCC: now also U9.39 (VSYS)
- net Y2R: now also U9.7 (GPIO5)
- net Y2W: now also U9.6 (GPIO4)
- new net: Q1.2 (B), R13.2
- new net: D4.2 (A), R14.1
- new net: Q1.1 (E), R14.2
- new net +5V: Q1.3 (C)
- no-connect marks 4 -> 0
Other:
- moved on the sheet: J3, R12, R18
