File: circuit/memory2.kicad_sch (KiCad schematic)
At the start: 20 parts, among them J2 Port C, J3 Port E, J4 Port A, J43 Port G, J5 Port D, U14 4081, U15 74LS32, U19 74HCT04, U2 74HTC175, U4 74LS32, U5 74HCT04

Commit message: .
Parts:
- removed U19: 74HCT04, symbol 74xx:74HCT04
- removed unit 3 of U5
- removed unit 6 of U5
- removed unit 5 of U5
- added C?: 10uF, symbol Device:C
Connections:
- net A16: now also J43.4 (Pin_4)
- net A17: now also J43.5 (Pin_5)
- net A18: now also J43.6 (Pin_6)
- net GND: now also C?.2
- net RAMONLY: now also J43.3 (Pin_3)
- net VCC: now also C?.1
Other:
- moved on the sheet: U14A, U14B, U14C, U14D, U15A, U15B, U5A, U5B

Commit message: .
Parts:
- added R? (x2): 10K, symbol Device:R_US
Connections:
- net RST: now also R?.1
- net VCC: now also R?.2, R?.2
- net ~{Y0W}: now also R?.1
Other:
- note added: "74HC04 (not)"
- note added: "74HC175 (flipflop)"
- note added: "74HC32 (or)"
- note added: "BIOS"
- note added: "CD4081 (and)"
- moved on the sheet: J2, J3, J4, J43, J5, U2, U?D

Commit message: .
Parts:
- added J1: Port B, symbol Connector_Generic:Conn_01x10
Connections:
- new net CLK_EXT: J1.9 (Pin_9)
- new net Y0R: J1.2 (Pin_2)
- new net Y0W: J1.1 (Pin_1)
- new net Y1R: J1.4 (Pin_4)
- new net Y1W: J1.3 (Pin_3)
- new net Y2R: J1.6 (Pin_6)
- new net Y2W: J1.5 (Pin_5)
- new net Y3R: J1.8 (Pin_8)
- new net Y3W: J1.7 (Pin_7)
- new net ~{WAIT}: J1.10 (Pin_10)
Changed lines of the file:
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@@
+    (stroke (width 0) (type default))
+  )
+  (wire (pts (xy 219.075 131.445) (xy 229.87 131.445))
     (stroke (width 0) (type default))
   )
@@
     (stroke (width 0) (type default))
   )
+  (wire (pts (xy 219.075 136.525) (xy 229.87 136.525))
+    (stroke (width 0) (type default))
+  )
   (wire (pts (xy 194.31 60.325) (xy 195.58 60.325))
     (stroke (width 0) (type default))
@@
     (stroke (width 0) (type default))
   )
+  (wire (pts (xy 219.075 123.825) (xy 229.87 123.825))
+    (stroke (width 0) (type default))
+  )
   (bus (pts (xy 34.925 40.005) (xy 34.925 37.465))
     (stroke (width 0) (type default))
@@
     (stroke (width 0) (type default))
   )
+  (wire (pts (xy 219.075 121.285) (xy 229.87 121.285))
+    (stroke (width 0) (type default))
+  )
   (bus (pts (xy 125.095 51.435) (xy 125.095 48.895))
     (stroke (width 0) (type default))
@@
     (stroke (width 0) (type default))
   )
+  (wire (pts (xy 219.075 128.905) (xy 229.87 128.905))
+    (stroke (width 0) (type default))
+  )
   (wire (pts (xy 272.415 131.445) (xy 261.62 131.445))
     (stroke (width 0) (type default))
@@
     (stroke (width 0) (type default))
   )
+  (wire (pts (xy 219.075 113.665) (xy 229.87 113.665))
+    (stroke (width 0) (type default))
+  )
   (wire (pts (xy 210.82 50.165) (xy 218.44 50.165))
     (stroke (width 0) (type default))
@@
     (stroke (width 0) (type default))
   )
+  (wire (pts (xy 219.075 126.365) (xy 229.87 126.365))
+    (stroke (width 0) (type default))
+  )
   (wire (pts (xy 272.415 133.985) (xy 261.62 133.985))
     (stroke (width 0) (type default))
   )
+  (wire (pts (xy 219.075 133.985) (xy 229.87 133.985))
+    (stroke (width 0) (type default))
+  )
   (bus (pts (xy 34.925 52.705) (xy 34.925 50.165))
     (stroke (width 0) (type default))
@@
     (stroke (width 0) (type default))
   )
+  (wire (pts (xy 219.075 116.205) (xy 229.87 116.205))
+    (stroke (width 0) (type default))
+  )
   (wire (pts (xy 132.08 137.795) (xy 135.89 137.795))
     (stroke (width 0) (type default))
@@
   )
   (wire (pts (xy 114.3 135.255) (xy 114.3 150.495))
+    (stroke (width 0) (type default))
+  )
+  (wire (pts (xy 219.075 118.745) (xy 229.87 118.745))
     (stroke (width 0) (type default))
   )
@@
     (effects (font (size 1.27 1.27)) (justify left bottom))
   )
+  (label "Y1R" (at 219.075 121.285 0) (fields_autoplaced)
+    (effects (font (size 1.27 1.27)) (justify left bottom))
+  )
+  (label "Y1W" (at 219.075 118.745 0) (fields_autoplaced)
+    (effects (font (size 1.27 1.27)) (justify left bottom))
+  )
   (label "A12" (at 272.415 156.21 180) (fields_autoplaced)
     (effects (font (size 1.27 1.27)) (justify right bottom))
@@
     (effects (font (size 1.27 1.27)) (justify left bottom))
   )
+  (label "Y3R" (at 219.075 131.445 0) (fields_autoplaced)
+    (effects (font (size 1.27 1.27)) (justify left bottom))
+  )
   (label "RAMONLY" (at 91.44 123.825 0) (fields_autoplaced)
     (effects (font (size 1.27 1.27)) (justify left bottom))
@@
     (effects (font (size 1.27 1.27)) (justify left bottom))
   )
+  (label "CLK_EXT" (at 219.075 133.985 0) (fields_autoplaced)
+    (effects (font (size 1.27 1.27)) (justify left bottom))
+  )
   (label "TX" (at 271.78 95.885 180) (fields_autoplaced)
     (effects (font (size 1.27 1.27)) (justify right bottom))
@@
     (effects (font (size 1.27 1.27)) (justify left bottom))
   )
+  (label "Y0R" (at 219.075 116.205 0) (fields_autoplaced)
+    (effects (font (size 1.27 1.27)) (justify left bottom))
+  )
   (label "D7" (at 272.415 131.445 180) (fields_autoplaced)
     (effects (font (size 1.27 1.27)) (justify right bottom))
   )
+  (label "~{WAIT}" (at 219.075 136.525 0) (fields_autoplaced)
+    (effects (font (size 1.27 1.27)) (justify left bottom))
+  )
   (label "~{WR}" (at 218.44 146.05 0) (fields_autoplaced)
     (effects (font (size 1.27 1.27)) (justify left bottom))
@@
     (effects (font (size 1.27 1.27)) (justify left bottom))
   )
+  (label "Y2R" (at 219.075 126.365 0) (fields_autoplaced)
+    (effects (font (size 1.27 1.27)) (justify left bottom))
+  )
   (label "A6" (at 218.44 161.29 0) (fields_autoplaced)
     (effects (font (size 1.27 1.27)) (justify left bottom))
@@
     (effects (font (size 1.27 1.27)) (justify left bottom))
   )
+  (label "Y2W" (at 219.075 123.825 0) (fields_autoplaced)
+    (effects (font (size 1.27 1.27)) (justify left bottom))
+  )
   (label "A18" (at 141.605 173.99 180) (fields_autoplaced)
     (effects (font (size 1.27 1.27)) (justify right bottom))
@@
     (effects (font (size 1.27 1.27)) (justify right bottom))
   )
+  (label "Y0W" (at 219.075 113.665 0) (fields_autoplaced)
+    (effects (font (size 1.27 1.27)) (justify left bottom))
+  )
   (label "RST" (at 172.085 67.945 0) (fields_autoplaced)
     (effects (font (size 1.27 1.27)) (justify left bottom))
@@
   (label "REG_A16" (at 255.27 40.005 180) (fields_autoplaced)
     (effects (font (size 1.27 1.27)) (justify right bottom))
+  )
+  (label "Y3W" (at 219.075 128.905 0) (fields_autoplaced)
+    (effects (font (size 1.27 1.27)) (justify left bottom))
   )
   (label "RX" (at 271.78 93.345 180) (fields_autoplaced)
@@
         )
       )
+    )
+  )
+  (symbol (lib_id "Connector_Generic:Conn_01x10") (at 234.95 123.825 0) (unit 1)
+    (in_bom yes) (on_board yes) (dnp no) (fields_autoplaced)
+    (property "Reference" "J1" (at 238.125 123.825 0)
+      (effects (font (size 1.27 1.27)) (justify left))
+    )
+    (property "Value" "Port B" (at 238.125 126.365 0)
+      (effects (font (size 1.27 1.27)) (justify left))
+    )
+    (property "Footprint" "" (at 234.95 123.825 0)
+      (effects (font (size 1.27 1.27)) hide)
+    )
+    (property "Datasheet" "~" (at 234.95 123.825 0)
+      (effects (font (size 1.27 1.27)) hide)
+    )
+    (pin "1")
+    (pin "10")
+    (pin "2")
+    (pin "3")
+    (pin "4")
+    (pin "5")
+    (pin "6")
+    (pin "7")
+    (pin "8")
+    (pin "9")
+    (instances
+      (project "fortuna-box"
+        (path "/0e4c4e8a-78e0-4f49-88dc-754c12656209"
+          (reference "J1") (unit 1)
+        )
+        (path "/0e4c4e8a-78e0-4f49-88dc-754c12656209/9a1861e1-3c11-472c-8fe5-ac282332e2ba"
+          (reference "J6") (unit 1)
+        )
+      )

Commit message: .
Connections:
- net RAMONLY: now also U2.14 (~{Q3}); no longer U2.15 (Q3)
Changed lines of the file:
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@@
   (junction (at 114.3 135.255) (diameter 0) (color 0 0 0 0)
   )
+  (no_connect (at 243.84 55.245))
+  (no_connect (at 243.84 47.625))
+  (no_connect (at 243.84 42.545))
   (no_connect (at 243.84 52.705))
-  (no_connect (at 243.84 47.625))
-  (no_connect (at 243.84 57.785))
-  (no_connect (at 243.84 42.545))
   (bus_entry (at 34.925 47.625) (size 2.54 2.54)
     (stroke (width 0) (type default))
@@
     (stroke (width 0) (type default))
   )
+  (wire (pts (xy 243.84 57.785) (xy 255.27 57.785))
+    (stroke (width 0) (type default))
+  )
   (bus (pts (xy 34.925 45.085) (xy 34.925 42.545))
     (stroke (width 0) (type default))
@@
   )
   (wire (pts (xy 255.27 50.165) (xy 243.84 50.165))
-    (stroke (width 0) (type default))
-  )
-  (wire (pts (xy 243.84 55.245) (xy 255.27 55.245))
     (stroke (width 0) (type default))
   )
@@
     (effects (font (size 1.27 1.27)) (justify left bottom))
   )
-  (label "RAMONLY" (at 255.27 55.245 180) (fields_autoplaced)
-    (effects (font (size 1.27 1.27)) (justify right bottom))
-  )
   (label "REG_A16" (at 92.075 155.575 0) (fields_autoplaced)
     (effects (font (size 1.27 1.27)) (justify left bottom))
@@
     (effects (font (size 1.27 1.27)) (justify right bottom))
   )
+  (label "RAMONLY" (at 255.27 57.785 180) (fields_autoplaced)
+    (effects (font (size 1.27 1.27)) (justify right bottom))
+  )

Commit message: .
Connections:
- net RAMONLY renamed ~{RAMONLY}
Changed lines of the file:
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@@
   (junction (at 114.3 135.255) (diameter 0) (color 0 0 0 0)
   )
+  (no_connect (at 243.84 52.705))
   (no_connect (at 243.84 55.245))
   (no_connect (at 243.84 47.625))
   (no_connect (at 243.84 42.545))
-  (no_connect (at 243.84 52.705))
   (bus_entry (at 34.925 47.625) (size 2.54 2.54)
     (stroke (width 0) (type default))
@@
     (stroke (width 0) (type default))
   )
+  (bus (pts (xy 34.925 45.085) (xy 34.925 42.545))
+    (stroke (width 0) (type default))
+  )
+  (wire (pts (xy 71.12 101.6) (xy 71.12 111.125))
+    (stroke (width 0) (type default))
+  )
+  (wire (pts (xy 106.045 79.375) (xy 119.38 79.375))
+    (stroke (width 0) (type default))
+  )
+  (bus (pts (xy 34.925 67.945) (xy 34.925 65.405))
+    (stroke (width 0) (type default))
+  )
+  (wire (pts (xy 82.55 81.915) (xy 82.55 67.945))
+    (stroke (width 0) (type default))
+  )
+  (wire (pts (xy 231.14 70.485) (xy 231.14 73.025))
+    (stroke (width 0) (type default))
+  )
+  (bus (pts (xy 150.495 53.975) (xy 150.495 51.435))
+    (stroke (width 0) (type default))
+  )
+  (wire (pts (xy 92.075 176.53) (xy 116.84 176.53))
+    (stroke (width 0) (type default))
+  )
+  (wire (pts (xy 272.415 153.67) (xy 261.62 153.67))
+    (stroke (width 0) (type default))
+  )
+  (wire (pts (xy 194.31 43.18) (xy 194.31 45.72))
+    (stroke (width 0) (type default))
+  )
+  (wire (pts (xy 62.865 65.405) (xy 74.93 65.405))
+    (stroke (width 0) (type default))
+  )
+  (wire (pts (xy 20.955 78.105) (xy 37.465 78.105))
+    (stroke (width 0) (type default))
+  )
+  (wire (pts (xy 132.08 163.195) (xy 141.605 163.195))
+    (stroke (width 0) (type default))
+  )
+  (wire (pts (xy 210.82 40.005) (xy 218.44 40.005))
+    (stroke (width 0) (type default))
+  )
+  (bus (pts (xy 65.405 52.705) (xy 65.405 50.165))
+    (stroke (width 0) (type default))
+  )
+  (wire (pts (xy 91.44 132.715) (xy 97.155 132.715))
+    (stroke (width 0) (type default))
+  )
+  (wire (pts (xy 62.865 67.945) (xy 82.55 67.945))
+    (stroke (width 0) (type default))
+  )
+  (wire (pts (xy 82.55 81.915) (xy 127.635 81.915))
+    (stroke (width 0) (type default))
+  )
+  (bus (pts (xy 125.095 66.675) (xy 125.095 64.135))
+    (stroke (width 0) (type default))
+  )
+  (bus (pts (xy 34.925 60.325) (xy 34.925 57.785))
+    (stroke (width 0) (type default))
+  )
+  (wire (pts (xy 78.105 101.6) (xy 78.105 111.125))
+    (stroke (width 0) (type default))
+  )
+  (bus (pts (xy 125.095 48.895) (xy 125.095 46.355))
+    (stroke (width 0) (type default))
+  )
+  (bus (pts (xy 125.095 59.055) (xy 125.095 56.515))
+    (stroke (width 0) (type default))
+  )
+  (bus (pts (xy 125.095 61.595) (xy 125.095 59.055))
+    (stroke (width 0) (type default))
+  )
+  (wire (pts (xy 255.27 45.085) (xy 243.84 45.085))
+    (stroke (width 0) (type default))
+  )
+  (wire (pts (xy 271.78 95.885) (xy 260.985 95.885))
+    (stroke (width 0) (type default))
+  )
+  (wire (pts (xy 173.99 135.255) (xy 173.99 142.875))
+    (stroke (width 0) (type default))
+  )
+  (bus (pts (xy 34.925 55.245) (xy 34.925 52.705))
+    (stroke (width 0) (type default))
+  )
+  (wire (pts (xy 272.415 161.29) (xy 261.62 161.29))
+    (stroke (width 0) (type default))
+  )
+  (wire (pts (xy 170.815 135.255) (xy 173.99 135.255))
+    (stroke (width 0) (type default))
+  )
+  (bus (pts (xy 65.405 40.005) (xy 65.405 37.465))
+    (stroke (width 0) (type default))
+  )
+  (wire (pts (xy 91.44 137.795) (xy 97.155 137.795))
+    (stroke (width 0) (type default))
+  )
+  (wire (pts (xy 272.415 148.59) (xy 261.62 148.59))
+    (stroke (width 0) (type default))
+  )
+  (wire (pts (xy 272.415 118.745) (xy 261.62 118.745))
+    (stroke (width 0) (type default))
+  )
+  (wire (pts (xy 20.955 73.025) (xy 37.465 73.025))
+    (stroke (width 0) (type default))
+  )
+  (bus (pts (xy 65.405 37.465) (xy 71.755 37.465))
+    (stroke (width 0) (type default))
+  )
   (wire (pts (xy 243.84 57.785) (xy 255.27 57.785))
-    (stroke (width 0) (type default))
-  )
-  (bus (pts (xy 34.925 45.085) (xy 34.925 42.545))
-    (stroke (width 0) (type default))
-  )
-  (wire (pts (xy 71.12 101.6) (xy 71.12 111.125))
-    (stroke (width 0) (type default))
-  )
-  (wire (pts (xy 106.045 79.375) (xy 119.38 79.375))
-    (stroke (width 0) (type default))
-  )
-  (bus (pts (xy 34.925 67.945) (xy 34.925 65.405))
-    (stroke (width 0) (type default))
-  )
-  (wire (pts (xy 82.55 81.915) (xy 82.55 67.945))
-    (stroke (width 0) (type default))
-  )
-  (wire (pts (xy 231.14 70.485) (xy 231.14 73.025))
-    (stroke (width 0) (type default))
-  )
-  (bus (pts (xy 150.495 53.975) (xy 150.495 51.435))
-    (stroke (width 0) (type default))
-  )
-  (wire (pts (xy 92.075 176.53) (xy 116.84 176.53))
-    (stroke (width 0) (type default))
-  )
-  (wire (pts (xy 272.415 153.67) (xy 261.62 153.67))
-    (stroke (width 0) (type default))
-  )
-  (wire (pts (xy 194.31 43.18) (xy 194.31 45.72))
-    (stroke (width 0) (type default))
-  )
-  (wire (pts (xy 62.865 65.405) (xy 74.93 65.405))
-    (stroke (width 0) (type default))
-  )
-  (wire (pts (xy 20.955 78.105) (xy 37.465 78.105))
-    (stroke (width 0) (type default))
-  )
-  (wire (pts (xy 132.08 163.195) (xy 141.605 163.195))
-    (stroke (width 0) (type default))
-  )
-  (wire (pts (xy 210.82 40.005) (xy 218.44 40.005))
-    (stroke (width 0) (type default))
-  )
-  (bus (pts (xy 65.405 52.705) (xy 65.405 50.165))
-    (stroke (width 0) (type default))
-  )
-  (wire (pts (xy 91.44 132.715) (xy 97.155 132.715))
-    (stroke (width 0) (type default))
-  )
-  (wire (pts (xy 62.865 67.945) (xy 82.55 67.945))
-    (stroke (width 0) (type default))
-  )
-  (wire (pts (xy 82.55 81.915) (xy 127.635 81.915))
-    (stroke (width 0) (type default))
-  )
-  (bus (pts (xy 125.095 66.675) (xy 125.095 64.135))
-    (stroke (width 0) (type default))
-  )
-  (bus (pts (xy 34.925 60.325) (xy 34.925 57.785))
-    (stroke (width 0) (type default))
-  )
-  (wire (pts (xy 78.105 101.6) (xy 78.105 111.125))
-    (stroke (width 0) (type default))
-  )
-  (bus (pts (xy 125.095 48.895) (xy 125.095 46.355))
-    (stroke (width 0) (type default))
-  )
-  (bus (pts (xy 125.095 59.055) (xy 125.095 56.515))
-    (stroke (width 0) (type default))
-  )
-  (bus (pts (xy 125.095 61.595) (xy 125.095 59.055))
-    (stroke (width 0) (type default))
-  )
-  (wire (pts (xy 255.27 45.085) (xy 243.84 45.085))
-    (stroke (width 0) (type default))
-  )
-  (wire (pts (xy 271.78 95.885) (xy 260.985 95.885))
-    (stroke (width 0) (type default))
-  )
-  (wire (pts (xy 173.99 135.255) (xy 173.99 142.875))
-    (stroke (width 0) (type default))
-  )
-  (bus (pts (xy 34.925 55.245) (xy 34.925 52.705))
-    (stroke (width 0) (type default))
-  )
-  (wire (pts (xy 272.415 161.29) (xy 261.62 161.29))
-    (stroke (width 0) (type default))
-  )
-  (wire (pts (xy 170.815 135.255) (xy 173.99 135.255))
-    (stroke (width 0) (type default))
-  )
-  (bus (pts (xy 65.405 40.005) (xy 65.405 37.465))
-    (stroke (width 0) (type default))
-  )
-  (wire (pts (xy 91.44 137.795) (xy 97.155 137.795))
-    (stroke (width 0) (type default))
-  )
-  (wire (pts (xy 272.415 148.59) (xy 261.62 148.59))
-    (stroke (width 0) (type default))
-  )
-  (wire (pts (xy 272.415 118.745) (xy 261.62 118.745))
-    (stroke (width 0) (type default))
-  )
-  (wire (pts (xy 20.955 73.025) (xy 37.465 73.025))
-    (stroke (width 0) (type default))
-  )
-  (bus (pts (xy 65.405 37.465) (xy 71.755 37.465))
     (stroke (width 0) (type default))
   )
@@
     (effects (font (size 1.27 1.27)) (justify left bottom))
   )
+  (label "~{RAMONLY}" (at 271.78 98.425 180) (fields_autoplaced)
+    (effects (font (size 1.27 1.27)) (justify right bottom))
+  )
   (label "Y1W" (at 219.075 118.745 0) (fields_autoplaced)
     (effects (font (size 1.27 1.27)) (justify left bottom))
@@
     (effects (font (size 1.27 1.27)) (justify left bottom))
   )
-  (label "RAMONLY" (at 91.44 123.825 0) (fields_autoplaced)
-    (effects (font (size 1.27 1.27)) (justify left bottom))
-  )
   (label "~{ROM_WE}" (at 218.44 153.67 0) (fields_autoplaced)
     (effects (font (size 1.27 1.27)) (justify left bottom))
@@
     (effects (font (size 1.27 1.27)) (justify right bottom))
   )
-  (label "RAMONLY" (at 255.27 57.785 180) (fields_autoplaced)
-    (effects (font (size 1.27 1.27)) (justify right bottom))
-  )
-  (label "RAMONLY" (at 271.78 98.425 180) (fields_autoplaced)
-    (effects (font (size 1.27 1.27)) (justify right bottom))
-  )
   (label "A18" (at 271.78 106.045 180) (fields_autoplaced)
     (effects (font (size 1.27 1.27)) (justify right bottom))
@@
     (effects (font (size 1.27 1.27)) (justify left bottom))
   )
+  (label "~{RAMONLY}" (at 99.695 123.825 180) (fields_autoplaced)
+    (effects (font (size 1.27 1.27)) (justify right bottom))
+  )
   (label "RX" (at 271.78 93.345 180) (fields_autoplaced)
     (effects (font (size 1.27 1.27)) (justify right bottom))
@@
     (effects (font (size 1.27 1.27)) (justify right bottom))
   )
+  (label "~{RAMONLY}" (at 255.27 57.785 180) (fields_autoplaced)
+    (effects (font (size 1.27 1.27)) (justify right bottom))
+  )
