File: circuit/memory2.kicad_sch (KiCad schematic)
At the start: 23 parts, among them J1 Port B, J2 Port C, J3 Port E, J4 Port A, J43 Port G, J5 Port D, U14 4081, U15 74LS32, U2 74HTC175, U4 74LS32, U5 74HCT04

Commit message: .
Parts:
- added J14: Port F, symbol Connector_Generic:Conn_01x08
Connections:
- net ~{RAMONLY}: no longer J43.3 (Pin_3)
- new net CLK: J14.7 (Pin_7)
- new net CLK_ENA: J14.8 (Pin_8)
- new net RAMONLY: J14.6 (Pin_6)
- new net ~{BUSAK}: J14.3 (Pin_3)
- new net ~{BUSRQ}: J14.2 (Pin_2)
- new net ~{IORQ}: J43.3 (Pin_3)
- new net ~{M1}: J14.5 (Pin_5)
- new net ~{NMI}: J14.4 (Pin_4)
- no-connect marks 4 -> 5
Changed lines of the file:
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@@
   (no_connect (at 243.84 52.705))
   (no_connect (at 243.84 55.245))
+  (no_connect (at 261.62 171.45))
   (no_connect (at 243.84 47.625))
   (no_connect (at 243.84 42.545))
@@
     (stroke (width 0) (type default))
   )
+  (wire (pts (xy 272.415 173.99) (xy 261.62 173.99))
+    (stroke (width 0) (type default))
+  )
   (wire (pts (xy 182.245 67.945) (xy 182.245 64.77))
     (stroke (width 0) (type default))
@@
     (stroke (width 0) (type default))
   )
+  (wire (pts (xy 272.415 176.53) (xy 261.62 176.53))
+    (stroke (width 0) (type default))
+  )
   (wire (pts (xy 219.075 121.285) (xy 229.87 121.285))
     (stroke (width 0) (type default))
@@
     (stroke (width 0) (type default))
   )
+  (wire (pts (xy 272.415 189.23) (xy 261.62 189.23))
+    (stroke (width 0) (type default))
+  )
   (wire (pts (xy 272.415 123.825) (xy 261.62 123.825))
     (stroke (width 0) (type default))
@@
     (stroke (width 0) (type default))
   )
+  (wire (pts (xy 272.415 181.61) (xy 261.62 181.61))
+    (stroke (width 0) (type default))
+  )
   (wire (pts (xy 272.415 161.29) (xy 261.62 161.29))
     (stroke (width 0) (type default))
@@
     (stroke (width 0) (type default))
   )
+  (wire (pts (xy 272.415 186.69) (xy 261.62 186.69))
+    (stroke (width 0) (type default))
+  )
   (wire (pts (xy 210.82 45.085) (xy 218.44 45.085))
     (stroke (width 0) (type default))
@@
     (stroke (width 0) (type default))
   )
+  (wire (pts (xy 272.415 184.15) (xy 261.62 184.15))
+    (stroke (width 0) (type default))
+  )
   (bus (pts (xy 125.095 41.275) (xy 125.095 38.735))
     (stroke (width 0) (type default))
@@
     (stroke (width 0) (type default))
   )
+  (wire (pts (xy 272.415 179.07) (xy 261.62 179.07))
+    (stroke (width 0) (type default))
+  )
   (wire (pts (xy 194.31 53.34) (xy 194.31 60.325))
     (stroke (width 0) (type default))
@@
     (fill (type none))
   )
-  (rectangle (start 208.28 82.55) (end 280.035 167.64)
+  (rectangle (start 208.28 82.55) (end 280.035 193.04)
     (stroke (width 0) (type default))
     (fill (type none))
@@
     (effects (font (size 1.27 1.27)) (justify left bottom))
   )
-  (label "~{RAMONLY}" (at 271.78 98.425 180) (fields_autoplaced)
+  (label "~{IORQ}" (at 271.78 98.425 180) (fields_autoplaced)
     (effects (font (size 1.27 1.27)) (justify right bottom))
   )
@@
     (effects (font (size 1.27 1.27)) (justify left bottom))
   )
+  (label "~{BUSRQ}" (at 272.415 173.99 180) (fields_autoplaced)
+    (effects (font (size 1.27 1.27)) (justify right bottom))
+  )
   (label "A12" (at 272.415 156.21 180) (fields_autoplaced)
     (effects (font (size 1.27 1.27)) (justify right bottom))
@@
     (effects (font (size 1.27 1.27)) (justify left bottom))
   )
+  (label "CLK_ENA" (at 272.415 189.23 180) (fields_autoplaced)
+    (effects (font (size 1.27 1.27)) (justify right bottom))
+  )
   (label "REG_A18" (at 92.075 176.53 0) (fields_autoplaced)
     (effects (font (size 1.27 1.27)) (justify left bottom))
@@
     (effects (font (size 1.27 1.27)) (justify left bottom))
   )
+  (label "~{BUSAK}" (at 272.415 176.53 180) (fields_autoplaced)
+    (effects (font (size 1.27 1.27)) (justify right bottom))
+  )
+  (label "CLK" (at 272.415 186.69 180) (fields_autoplaced)
+    (effects (font (size 1.27 1.27)) (justify right bottom))
+  )
   (label "D7" (at 272.415 131.445 180) (fields_autoplaced)
     (effects (font (size 1.27 1.27)) (justify right bottom))
@@
     (effects (font (size 1.27 1.27)) (justify left bottom))
   )
+  (label "~{M1}" (at 272.415 181.61 180) (fields_autoplaced)
+    (effects (font (size 1.27 1.27)) (justify right bottom))
+  )
+  (label "~{NMI}" (at 272.415 179.07 180) (fields_autoplaced)
+    (effects (font (size 1.27 1.27)) (justify right bottom))
+  )
   (label "Y2R" (at 219.075 126.365 0) (fields_autoplaced)
     (effects (font (size 1.27 1.27)) (justify left bottom))
@@
   )
   (label "~{RAMONLY}" (at 255.27 57.785 180) (fields_autoplaced)
+    (effects (font (size 1.27 1.27)) (justify right bottom))
+  )
+  (label "RAMONLY" (at 272.415 184.15 180) (fields_autoplaced)
     (effects (font (size 1.27 1.27)) (justify right bottom))
   )
@@
         )
       )
+    )
+  )
+  (symbol (lib_id "Connector_Generic:Conn_01x08") (at 256.54 179.07 0) (mirror y) (unit 1)
+    (in_bom yes) (on_board yes) (dnp no)
+    (property "Reference" "J14" (at 254 179.07 0)
+      (effects (font (size 1.27 1.27)) (justify left))
+    )
+    (property "Value" "Port F" (at 254 181.61 0)
+      (effects (font (size 1.27 1.27)) (justify left))
+    )
+    (property "Footprint" "" (at 256.54 179.07 0)
+      (effects (font (size 1.27 1.27)) hide)
+    )
+    (property "Datasheet" "~" (at 256.54 179.07 0)
+      (effects (font (size 1.27 1.27)) hide)
+    )
+    (pin "1")
+    (pin "2")
+    (pin "3")
+    (pin "4")
+    (pin "5")
+    (pin "6")
+    (pin "7")
+    (pin "8")
+    (instances
+      (project "fortuna-box"
+        (path "/0e4c4e8a-78e0-4f49-88dc-754c12656209"
+          (reference "J14") (unit 1)
+        )
+        (path "/0e4c4e8a-78e0-4f49-88dc-754c12656209/afd1b413-de30-4838-bb16-3d0c9f3cd196"
+          (reference "J12") (unit 1)
+        )
+        (path "/0e4c4e8a-78e0-4f49-88dc-754c12656209/34f47b44-6e82-4397-9bc8-849df4113da9"
+          (reference "J13") (unit 1)
+        )
+        (path "/0e4c4e8a-78e0-4f49-88dc-754c12656209/9a1861e1-3c11-472c-8fe5-ac282332e2ba"
+          (reference "J51") (unit 1)
+        )
+      )

Commit message: .
Connections:
- net CLK_ENA: no longer names the net of J14.8 (Pin_8)
- no-connect marks 5 -> 6
Changed lines of the file:
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@@
   (no_connect (at 243.84 55.245))
   (no_connect (at 261.62 171.45))
+  (no_connect (at 261.62 189.23))
   (no_connect (at 243.84 47.625))
   (no_connect (at 243.84 42.545))
@@
     (stroke (width 0) (type default))
   )
-  (wire (pts (xy 272.415 189.23) (xy 261.62 189.23))
-    (stroke (width 0) (type default))
-  )
   (wire (pts (xy 272.415 123.825) (xy 261.62 123.825))
     (stroke (width 0) (type default))
@@
     (effects (font (size 1.27 1.27)) (justify left bottom))
   )
-  (label "CLK_ENA" (at 272.415 189.23 180) (fields_autoplaced)
-    (effects (font (size 1.27 1.27)) (justify right bottom))
-  )
   (label "REG_A18" (at 92.075 176.53 0) (fields_autoplaced)

Commit message: .
Parts:
- renumbered J5 to J32, J4 to J41, J43 to J42, J2 to J45, J3 to J46, J14 to J51, J1 to J6
Changed lines of the file:
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@@
   (symbol (lib_id "Connector_Generic:Conn_01x06") (at 234.95 98.425 0) (unit 1)
     (in_bom yes) (on_board yes) (dnp no) (fields_autoplaced)
-    (property "Reference" "J4" (at 238.125 98.425 0)
+    (property "Reference" "J41" (at 238.125 98.425 0)
       (effects (font (size 1.27 1.27)) (justify left))
     )
@@
     (instances
       (project "fortuna-box"
-        (path "/0e4c4e8a-78e0-4f49-88dc-754c12656209"
-          (reference "J4") (unit 1)
-        )
-        (path "/0e4c4e8a-78e0-4f49-88dc-754c12656209/afd1b413-de30-4838-bb16-3d0c9f3cd196"
-          (reference "J7") (unit 1)
-        )
         (path "/0e4c4e8a-78e0-4f49-88dc-754c12656209/9a1861e1-3c11-472c-8fe5-ac282332e2ba"
           (reference "J41") (unit 1)
@@
   (symbol (lib_id "Connector_Generic:Conn_01x08") (at 256.54 179.07 0) (mirror y) (unit 1)
     (in_bom yes) (on_board yes) (dnp no)
-    (property "Reference" "J14" (at 254 179.07 0)
+    (property "Reference" "J51" (at 254 179.07 0)
       (effects (font (size 1.27 1.27)) (justify left))
     )
@@
     (instances
       (project "fortuna-box"
-        (path "/0e4c4e8a-78e0-4f49-88dc-754c12656209"
-          (reference "J14") (unit 1)
-        )
-        (path "/0e4c4e8a-78e0-4f49-88dc-754c12656209/afd1b413-de30-4838-bb16-3d0c9f3cd196"
-          (reference "J12") (unit 1)
-        )
-        (path "/0e4c4e8a-78e0-4f49-88dc-754c12656209/34f47b44-6e82-4397-9bc8-849df4113da9"
-          (reference "J13") (unit 1)
-        )
         (path "/0e4c4e8a-78e0-4f49-88dc-754c12656209/9a1861e1-3c11-472c-8fe5-ac282332e2ba"
           (reference "J51") (unit 1)
@@
   (symbol (lib_id "Connector_Generic:Conn_01x10") (at 234.95 123.825 0) (unit 1)
     (in_bom yes) (on_board yes) (dnp no) (fields_autoplaced)
-    (property "Reference" "J1" (at 238.125 123.825 0)
+    (property "Reference" "J6" (at 238.125 123.825 0)
       (effects (font (size 1.27 1.27)) (justify left))
     )
@@
     (instances
       (project "fortuna-box"
-        (path "/0e4c4e8a-78e0-4f49-88dc-754c12656209"
-          (reference "J1") (unit 1)
-        )
         (path "/0e4c4e8a-78e0-4f49-88dc-754c12656209/9a1861e1-3c11-472c-8fe5-ac282332e2ba"
           (reference "J6") (unit 1)
@@
   (symbol (lib_id "Connector_Generic:Conn_01x08") (at 234.315 153.67 0) (unit 1)
     (in_bom yes) (on_board yes) (dnp no) (fields_autoplaced)
-    (property "Reference" "J5" (at 237.49 153.67 0)
+    (property "Reference" "J32" (at 237.49 153.67 0)
       (effects (font (size 1.27 1.27)) (justify left))
     )
@@
     (instances
       (project "fortuna-box"
-        (path "/0e4c4e8a-78e0-4f49-88dc-754c12656209"
-          (reference "J5") (unit 1)
-        )
         (path "/0e4c4e8a-78e0-4f49-88dc-754c12656209/9a1861e1-3c11-472c-8fe5-ac282332e2ba"
           (reference "J32") (unit 1)
@@
   (symbol (lib_id "Connector_Generic:Conn_01x06") (at 255.905 98.425 0) (mirror y) (unit 1)
     (in_bom yes) (on_board yes) (dnp no)
-    (property "Reference" "J43" (at 252.73 98.425 0)
+    (property "Reference" "J42" (at 252.73 98.425 0)
       (effects (font (size 1.27 1.27)) (justify left))
     )
@@
     (instances
       (project "fortuna-box"
-        (path "/0e4c4e8a-78e0-4f49-88dc-754c12656209"
-          (reference "J43") (unit 1)
-        )
-        (path "/0e4c4e8a-78e0-4f49-88dc-754c12656209/afd1b413-de30-4838-bb16-3d0c9f3cd196"
-          (reference "J33") (unit 1)
-        )
         (path "/0e4c4e8a-78e0-4f49-88dc-754c12656209/9a1861e1-3c11-472c-8fe5-ac282332e2ba"
           (reference "J42") (unit 1)
@@
   (symbol (lib_id "Connector_Generic:Conn_01x08") (at 256.54 153.67 0) (mirror y) (unit 1)
     (in_bom yes) (on_board yes) (dnp no)
-    (property "Reference" "J3" (at 254 153.67 0)
+    (property "Reference" "J46" (at 254 153.67 0)
       (effects (font (size 1.27 1.27)) (justify left))
     )
@@
     (instances
       (project "fortuna-box"
-        (path "/0e4c4e8a-78e0-4f49-88dc-754c12656209"
-          (reference "J3") (unit 1)
-        )
         (path "/0e4c4e8a-78e0-4f49-88dc-754c12656209/9a1861e1-3c11-472c-8fe5-ac282332e2ba"
           (reference "J46") (unit 1)
@@
   (symbol (lib_id "Connector_Generic:Conn_01x10") (at 256.54 123.825 0) (mirror y) (unit 1)
     (in_bom yes) (on_board yes) (dnp no)
-    (property "Reference" "J2" (at 253.365 123.825 0)
+    (property "Reference" "J45" (at 253.365 123.825 0)
       (effects (font (size 1.27 1.27)) (justify left))
     )
@@
     (instances
       (project "fortuna-box"
-        (path "/0e4c4e8a-78e0-4f49-88dc-754c12656209"
-          (reference "J2") (unit 1)
-        )
         (path "/0e4c4e8a-78e0-4f49-88dc-754c12656209/9a1861e1-3c11-472c-8fe5-ac282332e2ba"
           (reference "J45") (unit 1)
